File: hdw/Host_Board/LED_Display_Controller/Panel_Data_Level_Shifters.sch (KiCad schematic (older format))
At the start: 0 parts

Commit message: Added pages for external memory, and added base parts for a few pages
Parts:
- added U?: 74HC245, symbol 74xx:74HC245
Changed lines of the file:
@@
 $Descr A 11000 8500
 encoding utf-8
-Sheet 10 12
+Sheet 10 14
 Title ""
 Date ""
@@
 Comment4 ""
 $EndDescr
+$Comp
+L 74xx:74HC245 U?
+U 1 1 5BAD6BC6
+P 4650 3530
+F 0 "U?" H 4350 4180 50  0000 C CNN
+F 1 "74HC245" H 4350 2880 50  0000 C CNN
+F 2 "" H 4650 3530 50  0001 C CNN
+F 3 "http://www.ti.com/lit/gpn/sn74HC245" H 4650 3530 50  0001 C CNN
+	1    4650 3530
+	1    0    0    -1
+$EndComp
 $EndSCHEMATC

Commit message: Changed panel data level shifter
Parts:
- removed U?: 74HC245, symbol 74xx:74HC245
- added U?: 74HC244, symbol 74xx:74HC244
Changed lines of the file:
@@
 $EndDescr
 $Comp
-L 74xx:74HC245 U?
-U 1 1 5BAD6BC6
-P 4650 3530
-F 0 "U?" H 4350 4180 50  0000 C CNN
-F 1 "74HC245" H 4350 2880 50  0000 C CNN
-F 2 "" H 4650 3530 50  0001 C CNN
-F 3 "http://www.ti.com/lit/gpn/sn74HC245" H 4650 3530 50  0001 C CNN
-	1    4650 3530
+L 74xx:74HC244 U?
+U 1 1 5BAD396C
+P 5520 3420
+F 0 "U?" H 5220 4070 50  0000 C CNN
+F 1 "74HC244" H 5220 2770 50  0000 C CNN
+F 2 "" H 5520 3420 50  0001 C CNN
+F 3 "http://www.nxp.com/documents/data_sheet/74HC_HCT244.pdf" H 5520 3420 50  0001 C CNN
+	1    5520 3420
 	1    0    0    -1
 $EndComp

Commit message: Changed output data buffer for thrid time
Parts:
- removed U?: 74HC244, symbol 74xx:74HC244
- added U?: 74HCT541, symbol 74xx:74HCT541
Changed lines of the file:
@@
 $EndDescr
 $Comp
-L 74xx:74HC244 U?
-U 1 1 5BAD396C
-P 5520 3420
-F 0 "U?" H 5220 4070 50  0000 C CNN
-F 1 "74HC244" H 5220 2770 50  0000 C CNN
-F 2 "" H 5520 3420 50  0001 C CNN
-F 3 "http://www.nxp.com/documents/data_sheet/74HC_HCT244.pdf" H 5520 3420 50  0001 C CNN
-	1    5520 3420
+L 74xx:74HCT541 U?
+U 1 1 5BAD3B80
+P 5510 3500
+F 0 "U?" H 5210 4150 50  0000 C CNN
+F 1 "74HCT541" H 5210 2850 50  0000 C CNN
+F 2 "" H 5510 3500 50  0001 C CNN
+F 3 "http://www.ti.com/lit/gpn/sn74HCT541" H 5510 3500 50  0001 C CNN
+	1    5510 3500
 	1    0    0    -1
 $EndComp

Commit message: added panel data conns
Parts:
- added J?: STRING_1, symbol Connector_Generic:Conn_02x08_Odd_Even
Connections:
- net labels added: A_POS5, B1_POS5, B2_POS5, B_POS5, CLK_POS5, C_POS5, D_POS5, E_POS5, G1_POS5, G2_POS5, GND, LAT_POS5, R1_POS5, R2_POS5, ~OE_POS5
- wire segments 0 -> 4
Changed lines of the file:
@@
 	1    0    0    -1
 $EndComp
+$Comp
+L Connector_Generic:Conn_02x08_Odd_Even J?
+U 1 1 5BB413E8
+P 1800 4550
+F 0 "J?" H 1850 5067 50  0000 C CNN
+F 1 "STRING_1" H 1850 4976 50  0000 C CNN
+F 2 "" H 1800 4550 50  0001 C CNN
+F 3 "~" H 1800 4550 50  0001 C CNN
+	1    1800 4550
+	1    0    0    -1
+$EndComp
+Text GLabel 1600 4650 0    50   Input ~ 0
+A_POS5
+Text GLabel 2100 4650 2    50   Input ~ 0
+B_POS5
+Text GLabel 2100 4750 2    50   Input ~ 0
+D_POS5
+Text GLabel 2100 4550 2    50   Input ~ 0
+E_POS5
+Text GLabel 1600 4750 0    50   Input ~ 0
+C_POS5
+Text GLabel 1600 4850 0    50   Input ~ 0
+CLK_POS5
+Text GLabel 1600 4950 0    40   Input ~ 0
+~OE_POS5
+Text GLabel 2100 4850 2    50   Input ~ 0
+LAT_POS5
+Text GLabel 1600 4250 0    50   Input ~ 0
+R1_POS5
+Text GLabel 1600 4350 0    50   Input ~ 0
+B1_POS5
+Text GLabel 1600 4450 0    50   Input ~ 0
+R2_POS5
+Text GLabel 1600 4550 0    50   Input ~ 0
+B2_POS5
+Text GLabel 2100 4250 2    50   Input ~ 0
+G1_POS5
+Text GLabel 2100 4450 2    50   Input ~ 0
+G2_POS5
+$Comp
+L power:GND #PWR?
+U 1 1 5BB413FD
+P 2650 5100
+F 0 "#PWR?" H 2650 4850 50  0001 C CNN
+F 1 "GND" H 2655 4927 50  0000 C CNN
+F 2 "" H 2650 5100 50  0001 C CNN
+F 3 "" H 2650 5100 50  0001 C CNN
+	1    2650 5100
+	1    0    0    -1
+$EndComp
+Wire Wire Line
+	2650 5100 2650 4950
+Wire Wire Line
+	2650 4950 2100 4950
+Wire Wire Line
+	2100 4350 2650 4350
+Wire Wire Line
+	2650 4350 2650 4950
+Connection ~ 2650 4950
 $EndSCHEMATC

Commit message: Added panel data level shifters pages
Parts:
- removed J?: STRING_1, symbol Connector_Generic:Conn_02x08_Odd_Even
- added J?: STRING_1, symbol Connector_Generic:Conn_02x08_Odd_Even
- added R? (x15): 10K, symbol LED_Display_Local_Library:R_Custom
- added R? (x12): 100, symbol LED_Display_Local_Library:R_Custom
Connections:
- net labels added: +3.3V, B1_POS3P3, B2_POS3P3, G1_POS3P3, G2_POS3P3, LVL_SHFT_EN, R1_POS3P3, R2_POS3P3
- wire segments 4 -> 50
- no-connect marks 0 -> 2
Other:
- moved on the sheet: U?
