File: hdw/Host_Board/LED_Display_Controller/Panel_Power_Connectors.sch (KiCad schematic (older format))
At the start: 0 parts

Commit message: Added panel power connectors (and updated pdf)
Parts:
- added J? (x40): Conn_01x01, symbol Connector_Generic:Conn_01x01

Commit message: fixed panel power connectors and added level shifters for A, B, C, D, E, CLK, LAT, OE
Parts:
- removed J? (x38): Conn_01x01, symbol Connector_Generic:Conn_01x01
- added C? (x20): C_Custom, symbol LED_Display_Local_Library:C_Custom
- added J? (x19): 5V_OUT, symbol Connector_Generic:Conn_01x01
- added J? (x19): GND_OUT, symbol Connector_Generic:Conn_01x01
- J?: value Conn_01x01 -> 5V_OUT
- J?: value Conn_01x01 -> GND_OUT
Connections:
- net labels added: +5V, GND
- wire segments 0 -> 40
