File: hdw/Host_Board/LED_Display_Controller/External_Flash_3.sch (KiCad schematic (older format))
At the start: 0 parts

Commit message: Wired Micro to external SRAM, copied Flash 8 times
Parts:
- added C?: 0.1uF, symbol LED_Display_Local_Library:C_Custom
- added C?: 10nF, symbol LED_Display_Local_Library:C_Custom
- added C?: 1nF, symbol LED_Display_Local_Library:C_Custom
- added J?: WP3, symbol Connector_Generic:Conn_02x01
- added R? (x6): 10k, symbol Custom_Library:R_Custom
- added R? (x5): 100, symbol Custom_Library:R_Custom
- added U?: SST25PF020B, Housings_SOIC:SOIC-8_3.9x4.9mm_Pitch1.27mm, symbol LED_Display_Local_Library:SST25PF020B
Connections:
- net labels added: +3.3V, FLASH_MISO, FLASH_MOSI, FLASH_SCK, GND, ~FLASH_CE3, ~FLASH_Hold
- wire segments 0 -> 30

Commit message: Added to-do list, cleaned some pages, ~MCLR filter
Parts:
- added R?: 100, symbol Custom_Library:R_Custom
Connections:
- net labels added: ~FLASH_WP3
- wire segments 30 -> 31
Changed lines of the file:
@@
 $Descr A 11000 8500
 encoding utf-8
-Sheet 18 25
+Sheet 16 25
 Title ""
 Date ""
@@
 AR Path="/5BB181D8/5BBE81C8" Ref="C?"  Part="1"
 AR Path="/5BB2595E/5BBE81C8" Ref="C?"  Part="1"
+AR Path="/5BB25AEA/5BBE81C8" Ref="C?"  Part="1"
 F 0 "C?" H 5815 5530 50  0000 L CNN
 F 1 "0.1uF" H 5815 5330 50  0000 L CNN
@@
 AR Path="/5BB181D8/5BBE81D3" Ref="C?"  Part="1"
 AR Path="/5BB2595E/5BBE81D3" Ref="C?"  Part="1"
+AR Path="/5BB25AEA/5BBE81D3" Ref="C?"  Part="1"
 F 0 "C?" H 6115 5530 50  0000 L CNN
 F 1 "10nF" H 6115 5330 50  0000 L CNN
@@
 AR Path="/5BB181D8/5BBE81DE" Ref="C?"  Part="1"
 AR Path="/5BB2595E/5BBE81DE" Ref="C?"  Part="1"
+AR Path="/5BB25AEA/5BBE81DE" Ref="C?"  Part="1"
 F 0 "C?" H 6415 5530 50  0000 L CNN
 F 1 "1nF" H 6415 5330 50  0000 L CNN
@@
 AR Path="/5BB181D8/5BBE81E5" Ref="#PWR?"  Part="1"
 AR Path="/5BB2595E/5BBE81E5" Ref="#PWR?"  Part="1"
+AR Path="/5BB25AEA/5BBE81E5" Ref="#PWR?"  Part="1"
 F 0 "#PWR?" H 6090 5410 50  0001 C CNN
 F 1 "GND" H 6090 5510 50  0000 C CNN
@@
 AR Path="/5BB181D8/5BBE81F2" Ref="#PWR?"  Part="1"
 AR Path="/5BB2595E/5BBE81F2" Ref="#PWR?"  Part="1"
+AR Path="/5BB25AEA/5BBE81F2" Ref="#PWR?"  Part="1"
 F 0 "#PWR?" H 6090 5050 50  0001 C CNN
 F 1 "+3.3V" H 6090 5340 50  0000 C CNN
@@
 Text GLabel 3270 3550 0    40   Input ~ 0
 ~FLASH_Hold
+$Comp
+L Custom_Library:R_Custom R?
+U 1 1 5BC1CF11
+P 3420 3650
+F 0 "R?" V 3380 3780 50  0000 L CNN
+F 1 "100" V 3420 3650 50  0000 C CNN
+F 2 "" H 3420 3650 50  0001 C CNN
+F 3 "" H 3420 3650 50  0001 C CNN
+F 4 "0603" V 3520 3650 50  0001 C CNN "display_footprint"
+F 5 "1%" V 3620 3650 50  0001 C CNN "Tolerance"
+F 6 "1/10W" V 3720 3650 50  0001 C CNN "Wattage"
+F 7 "PN" H 3720 4050 60  0001 C CNN "Digi-Key PN"
+	1    3420 3650
+	0    1    1    0
+$EndComp
+Wire Wire Line
+	3570 3650 3930 3650
+Text GLabel 3270 3650 0    40   Input ~ 0
+~FLASH_WP3
 $EndSCHEMATC
