File: hdw/Host_Board/LED_Display_Controller/POS5_Phase_1.sch (KiCad schematic (older format))
At the start: 0 parts

Commit message: Overriding master branch for clean pull request
Parts:
- added C? (x2): 1uF, Capacitors_SMD:C_0603, symbol LED_Display_Local_Library:C_Custom
- added C? (x2): 0.1uF, Capacitors_SMD:C_0603, symbol LED_Display_Local_Library:C_Custom
- added C?: 0.22uF, Capacitors_SMD:C_0603, symbol LED_Display_Local_Library:C_Custom
- added C? (x2): 22uF, Capacitors_SMD:C_1210, symbol LED_Display_Local_Library:C_Custom
- added C? (x2): 100uF, Capacitors_SMD:C_1210, symbol LED_Display_Local_Library:C_Custom
- added C?: 100uF, Capacitors_Tantalum_SMD:CP_Tantalum_Case-B_EIA-3528-21_Reflow, symbol LED_Display_Local_Library:CP_Tant_Custom
- added C?: 2200pF, Capacitors_SMD:C_0603, symbol LED_Display_Local_Library:C_Custom
- added C? (x3): 100pF, Capacitors_SMD:C_0603, symbol LED_Display_Local_Library:C_Custom
- added C?: 3300pF, Capacitors_SMD:C_0603, symbol LED_Display_Local_Library:C_Custom
- added L?: 0.47uH, Inductors_SMD:L_Vishay_IHLP-4040, symbol LED_Display_Local_Library:L_Custom
- added R? (x2): 2, Resistors_SMD:R_0603, symbol LED_Display_Local_Library:R_Custom
- added R?: 1.4k, Resistors_SMD:R_0603, symbol LED_Display_Local_Library:R_Custom
- added R? (x2): 0, Resistors_SMD:R_0603, symbol LED_Display_Local_Library:R_Custom
- added R?: 100k, Resistors_SMD:R_0603, symbol LED_Display_Local_Library:R_Custom
- added R?: 13.7k, Resistors_SMD:R_0603, symbol LED_Display_Local_Library:R_Custom
- added R?: 10k, Resistors_SMD:R_0603, symbol LED_Display_Local_Library:R_Custom
- added R?: 320, Resistors_SMD:R_0603, symbol LED_Display_Local_Library:R_Custom
- added R?: 6.04k, Resistors_SMD:R_0603, symbol LED_Display_Local_Library:R_Custom
- added R?: 66.5k, Resistors_SMD:R_0603, symbol LED_Display_Local_Library:R_Custom
- added U?: SiC779, Custom Footprints Library:MLP66-40_6x6mm_Pitch0.5mm, symbol LED_Display_Local_Library:SiC779
- added U?: LTC7851UHH, Custom Footprints Library:QFN-58-1EP_9x5mm_Pitch0.4mm, symbol LED_Display_Local_Library:LTC7851UHH
Connections:
- net labels added: +12V, +5.5V_MNG, +5V, GND, LOOP_TAP, POS5_COMP, POS5_IAVG, POS5_ILIM, POS5_ISNS1_+, POS5_ISNS1_-, POS5_PGOOD_OC, POS5_RUN, POS5_SS, POS5_VOSNS, POS5_VSNS1_+, POS5_VSNS1_-, ~POS5_THDN
- wire segments 0 -> 157
- no-connect marks 0 -> 3
Other:
- note added: "+5V Phase 1"
- note added: "Route as diff pairs"
