File: hdw/Host_Board/LED_Display_Controller/POS5P5_MNG.sch (KiCad schematic (older format))
At the start: 0 parts

Commit message: Overriding master branch for clean pull request
Parts:
- added C? (x3): 0.1uF, Capacitors_SMD:C_0603, symbol LED_Display_Local_Library:C_Custom
- added C?: 100uF, Capacitors_Tantalum_SMD:CP_Tantalum_Case-B_EIA-3528-21_Reflow, symbol LED_Display_Local_Library:CP_Tant_Custom
- added C?: 10uF, Capacitors_Tantalum_SMD:CP_Tantalum_Case-B_EIA-3528-21_Reflow, symbol LED_Display_Local_Library:CP_Tant_Custom
- added R?: 200, Resistors_SMD:R_0603, symbol LED_Display_Local_Library:R_Custom
- added R?: 680, Resistors_SMD:R_0603, symbol LED_Display_Local_Library:R_Custom
- added TP?: TP, Measurement_Points:Measurement_Point_Round-SMD-Pad_Small, symbol Custom_Library:TP
- added U?: LM1117-ADJ, TO_SOT_Packages_SMD:SOT-223-3_TabPin2, symbol Regulator_Linear:LM1117-ADJ
Connections:
- net labels added: +12V, +5.5V_MNG, GND
- wire segments 0 -> 18
Other:
- note added: "+5.5V MNG LDO"
