File: hdw/Host_Board/LED_Display_Controller/Internal_Rail_Monitoring.sch (KiCad schematic (older format))
At the start: 0 parts

Commit message: rage commit
Parts:
- added C? (x5): 330pF, symbol LED_Display_Local_Library:C_Custom
- added D? (x5): MM5Z3V3ST1G, Diode_SMD:D_SOD-523, symbol Diode:MM5Zxx
- added R? (x9): 10k, symbol Custom_Library:R_Custom
- added R?: 1k, symbol Custom_Library:R_Custom
Connections:
- new net +12V: R?.1
- new net +3V3: R?.1
- new net +5.5V: R?.1
- new net +5V: R?.1
- new net +5VP: R?.1
- new net GND: C?.2, C?.2, C?.2, C?.2, C?.2, D?.2 (A), D?.2 (A), D?.2 (A), D?.2 (A), D?.2 (A), R?.2, R?.2, R?.2, R?.2, R?.2
- new net POS12_ADC: C?.1, D?.1 (K), R?.1, R?.2
- new net POS3P3_ADC: C?.1, D?.1 (K), R?.1, R?.2
- new net POS5P5_ADC: C?.1, D?.1 (K), R?.1, R?.2
- new net POS5P_ADC: C?.1, D?.1 (K), R?.1, R?.2
- new net POS5_ADC: C?.1, D?.1 (K), R?.1, R?.2
Other:
- note added: "15. Internal Rail Monitoring"
