File: hdw/Host_Board/LED_Display_Controller/Mechanical.sch (KiCad schematic (older format))
At the start: 0 parts

Commit message: Added a few pages and edits
Parts:
- added H? (x12): 3mm Mounting Hole, symbol Mechanical:MountingHole
- added MK? (x12): 4-40 Standoff, symbol LED_Display_Local_Library:Standoff
- added MK? (x12): Screw, symbol LED_Display_Local_Library:Screw

Commit message: rage commit
Parts:
- MK? (x12): value Screw -> 4-40 Screw
Other:
- note added: "31. Mechanical"
- moved on the sheet: H?, MK?
