File: hdw/Host_Board/LED_Display_Controller/Panel_Data_Level_Shifters_1.sch (KiCad schematic (older format))
At the start: 62 parts

Commit message: I said never do this, it's bad for you
Connections:
- net +3V3: no longer C?.1, C?.1, C?.1, C?.1, C?.1, C?.1, U?.20 (VCC), U?.20 (VCC)
- new net +5V: C?.1, C?.1, C?.1, C?.1, C?.1, C?.1, U?.20 (VCC), U?.20 (VCC)
Changed lines of the file:
@@
 $Descr A 11000 8500
 encoding utf-8
-Sheet 23 32
+Sheet 22 31
 Title ""
 Date ""
@@
 G2_POS5
 $Comp
-L power:+3.3V #PWR?
-U 1 1 5BB6DBEF
-P 5500 1420
-AR Path="/5BAAE2B6/5BB6DBEF" Ref="#PWR?"  Part="1"
-AR Path="/5BB6CF6D/5BB6DBEF" Ref="#PWR?"  Part="1"
-AR Path="/5BBE424C/5BB6DBEF" Ref="#PWR?"  Part="1"
-F 0 "#PWR?" H 5500 1270 50  0001 C CNN
-F 1 "+3.3V" H 5500 1560 50  0000 C CNN
-F 2 "" H 5500 1420 50  0001 C CNN
-F 3 "" H 5500 1420 50  0001 C CNN
-	1    5500 1420
-	1    0    0    -1
-$EndComp
-$Comp
 L power:GND #PWR?
 U 1 1 5BB6DBF5
@@
 G4_POS5
 $Comp
-L power:+3.3V #PWR?
-U 1 1 5BB6EA78
-P 5500 3950
-AR Path="/5BAAE2B6/5BB6EA78" Ref="#PWR?"  Part="1"
-AR Path="/5BB6CF6D/5BB6EA78" Ref="#PWR?"  Part="1"
-AR Path="/5BBE424C/5BB6EA78" Ref="#PWR?"  Part="1"
-F 0 "#PWR?" H 5500 3800 50  0001 C CNN
-F 1 "+3.3V" H 5500 4090 50  0000 C CNN
-F 2 "" H 5500 3950 50  0001 C CNN
-F 3 "" H 5500 3950 50  0001 C CNN
-	1    5500 3950
-	1    0    0    -1
-$EndComp
-$Comp
 L power:GND #PWR?
 U 1 1 5BB6EA7E
@@
 Wire Wire Line
 	2870 3370 2870 3330
-$Comp
-L power:+3.3V #PWR?
-U 1 1 5BB8B9C0
-P 2570 2950
-AR Path="/5BAAE16C/5BB8B9C0" Ref="#PWR?"  Part="1"
-AR Path="/5BB6CF6D/5BB8B9C0" Ref="#PWR?"  Part="1"
-AR Path="/5BBE424C/5BB8B9C0" Ref="#PWR?"  Part="1"
-F 0 "#PWR?" H 2570 2800 50  0001 C CNN
-F 1 "+3.3V" H 2570 3090 50  0000 C CNN
-F 2 "" H 2570 2950 50  0001 C CNN
-F 3 "" H 2570 2950 50  0001 C CNN
-	1    2570 2950
-	1    0    0    -1
-$EndComp
 Wire Wire Line
 	2570 2950 2570 2990
@@
 Wire Wire Line
 	2870 5900 2870 5860
-$Comp
-L power:+3.3V #PWR?
-U 1 1 5BB8F3A4
+Wire Wire Line
+	2570 5480 2570 5520
+Wire Wire Line
+	2270 5560 2270 5520
+Wire Wire Line
+	2270 5520 2570 5520
+Wire Wire Line
+	2870 5520 2870 5560
+Connection ~ 2570 5520
+Wire Wire Line
+	2570 5520 2570 5560
+Wire Wire Line
+	2570 5520 2870 5520
+$Comp
+L power:+5V #PWR?
+U 1 1 5BF4791B
+P 5500 1420
+F 0 "#PWR?" H 5500 1270 50  0001 C CNN
+F 1 "+5V" H 5500 1560 50  0000 C CNN
+F 2 "" H 5500 1420 50  0001 C CNN
+F 3 "" H 5500 1420 50  0001 C CNN
+	1    5500 1420
+	1    0    0    -1
+$EndComp
+$Comp
+L power:+5V #PWR?
+U 1 1 5BF47ADF
+P 2570 2950
+F 0 "#PWR?" H 2570 2800 50  0001 C CNN
+F 1 "+5V" H 2570 3090 50  0000 C CNN
+F 2 "" H 2570 2950 50  0001 C CNN
+F 3 "" H 2570 2950 50  0001 C CNN
+	1    2570 2950
+	1    0    0    -1
+$EndComp
+$Comp
+L power:+5V #PWR?
+U 1 1 5BF47F46
+P 5500 3950
+F 0 "#PWR?" H 5500 3800 50  0001 C CNN
+F 1 "+5V" H 5500 4090 50  0000 C CNN
+F 2 "" H 5500 3950 50  0001 C CNN
+F 3 "" H 5500 3950 50  0001 C CNN
+	1    5500 3950
+	1    0    0    -1
+$EndComp
+$Comp
+L power:+5V #PWR?
+U 1 1 5BF480C5
 P 2570 5480
-AR Path="/5BAAE16C/5BB8F3A4" Ref="#PWR?"  Part="1"
-AR Path="/5BB6CF6D/5BB8F3A4" Ref="#PWR?"  Part="1"
-AR Path="/5BBE424C/5BB8F3A4" Ref="#PWR?"  Part="1"
 F 0 "#PWR?" H 2570 5330 50  0001 C CNN
-F 1 "+3.3V" H 2570 5620 50  0000 C CNN
+F 1 "+5V" H 2570 5620 50  0000 C CNN
 F 2 "" H 2570 5480 50  0001 C CNN
 F 3 "" H 2570 5480 50  0001 C CNN
@@
 	1    0    0    -1
 $EndComp
-Wire Wire Line
-	2570 5480 2570 5520
-Wire Wire Line
-	2270 5560 2270 5520
-Wire Wire Line
-	2270 5520 2570 5520
-Wire Wire Line
-	2870 5520 2870 5560
-Connection ~ 2570 5520
-Wire Wire Line
-	2570 5520 2570 5560
-Wire Wire Line
-	2570 5520 2870 5520
 $EndSCHEMATC

Commit message: rage commit
Other:
- note added: "26. Panel Data Level Shifters 1"
