File: hdw/Power_Board/LTC7851_Demo/Active_Load_1.sch (KiCad schematic (older format))
At the start: 16 parts, among them J1101 FG_LOAD, J1102 ISNS, Q1101 IPC100N04S51R7ATMA1, Q1102 IPC100N04S51R7ATMA1, U1101 LT1010DD

Commit message: Merging drews_branch_3 into master
Parts:
- C1101, C1102: symbol Custom_Library:C_Custom -> LED_Display_Local_Library:C_Custom
- C1103: symbol Custom_Library:CP_Tant_Custom -> LED_Display_Local_Library:CP_Tant_Custom
- R1101, R1102, R1103, R1104, R1105, R1106, R1107, R1108: symbol Custom_Library:R_Custom -> LED_Display_Local_Library:R_Custom
- U1101: symbol Custom_Library:LT1010DD -> LED_Display_Local_Library:LT1010DD
Other:
- note added: "11. Active Load Driver and Active Load Bank 1"
- note removed: "Active Load Driver and Active Load Bank 1"
Changed lines of the file:
@@
 $EndComp
 $Comp
-L Custom_Library:R_Custom R?
+L LED_Display_Local_Library:R_Custom R?
 U 1 1 5BC370E8
 P 8000 2940
@@
 $EndComp
 $Comp
-L Custom_Library:R_Custom R?
+L LED_Display_Local_Library:R_Custom R?
 U 1 1 5BC37C2E
 P 7240 2640
@@
 F 2 "Resistors_SMD:R_0603" H 7240 2640 50  0001 C CNN
 F 3 "" H 7240 2640 50  0001 C CNN
-F 4 "0603" H 7320 2720 50  0000 L CNN "display_footprint"
-F 5 "1%" H 7320 2640 50  0000 L CNN "Tolerance"
-F 6 "1/10W" H 7320 2560 50  0000 L CNN "Wattage"
-F 7 "RHM10KADCT-ND" H 7540 3040 60  0001 C CNN "Digi-Key PN"
+F 4 "RHM10KADCT-ND" H 7540 3040 60  0001 C CNN "Digi-Key PN"
+F 5 "0603" H 7320 2720 50  0000 L CNN "display_footprint"
+F 6 "1%" H 7320 2640 50  0000 L CNN "Tolerance"
+F 7 "1/10W" H 7320 2560 50  0000 L CNN "Wattage"
 	1    7240 2640
 	1    0    0    -1
@@
 	7240 2420 7700 2420
 $Comp
-L Custom_Library:R_Custom R1103
+L LED_Display_Local_Library:R_Custom R1103
 U 1 1 5BC37FB0
 P 6560 2420
@@
 F 2 "Resistors_SMD:R_0603" H 6560 2420 50  0001 C CNN
 F 3 "" H 6560 2420 50  0001 C CNN
-F 4 "0603" V 6660 2420 50  0000 C CNN "display_footprint"
-F 5 "1%" V 6760 2420 50  0000 C CNN "Tolerance"
-F 6 "1/10W" V 6860 2420 50  0000 C CNN "Wattage"
-F 7 "YAG3351CT-ND" H 6860 2820 60  0001 C CNN "Digi-Key PN"
+F 4 "YAG3351CT-ND" H 6860 2820 60  0001 C CNN "Digi-Key PN"
+F 5 "0603" V 6660 2420 50  0000 C CNN "display_footprint"
+F 6 "1%" V 6760 2420 50  0000 C CNN "Tolerance"
+F 7 "1/10W" V 6860 2420 50  0000 C CNN "Wattage"
 	1    6560 2420
 	0    1    1    0
@@
 LOAD_GATE
 $Comp
-L Custom_Library:LT1010DD U1101
+L LED_Display_Local_Library:LT1010DD U1101
 U 1 1 5BC3FE8E
 P 3160 3510
@@
 $EndComp
 $Comp
-L Custom_Library:R_Custom R?
+L LED_Display_Local_Library:R_Custom R?
 U 1 1 5BC405D3
 P 3260 2980
@@
 F 2 "Resistors_SMD:R_0603" H 3260 2980 50  0001 C CNN
 F 3 "" H 3260 2980 50  0001 C CNN
-F 4 "0603" H 3340 3060 50  0000 L CNN "display_footprint"
-F 5 "1%" H 3340 2980 50  0000 L CNN "Tolerance"
-F 6 "1/10W" H 3340 2900 50  0000 L CNN "Wattage"
-F 7 "YAG3351CT-ND" H 3560 3380 60  0001 C CNN "Digi-Key PN"
+F 4 "YAG3351CT-ND" H 3560 3380 60  0001 C CNN "Digi-Key PN"
+F 5 "0603" H 3340 3060 50  0000 L CNN "display_footprint"
+F 6 "1%" H 3340 2980 50  0000 L CNN "Tolerance"
+F 7 "1/10W" H 3340 2900 50  0000 L CNN "Wattage"
 	1    3260 2980
 	1    0    0    -1
@@
 	1950 3610 1870 3610
 $Comp
-L Custom_Library:R_Custom R?
+L LED_Display_Local_Library:R_Custom R?
 U 1 1 5BC41AD3
 P 2500 3730
@@
 F 2 "Resistors_SMD:R_0603" H 2500 3730 50  0001 C CNN
 F 3 "" H 2500 3730 50  0001 C CNN
-F 4 "0603" H 2580 3810 50  0000 L CNN "display_footprint"
-F 5 "1%" H 2580 3730 50  0000 L CNN "Tolerance"
-F 6 "1/10W" H 2580 3650 50  0000 L CNN "Wattage"
-F 7 "RHM10KADCT-ND" H 2800 4130 60  0001 C CNN "Digi-Key PN"
+F 4 "RHM10KADCT-ND" H 2800 4130 60  0001 C CNN "Digi-Key PN"
+F 5 "0603" H 2580 3810 50  0000 L CNN "display_footprint"
+F 6 "1%" H 2580 3730 50  0000 L CNN "Tolerance"
+F 7 "1/10W" H 2580 3650 50  0000 L CNN "Wattage"
 	1    2500 3730
 	-1   0    0    -1
@@
 $EndComp
 $Comp
-L Custom_Library:R_Custom R?
+L LED_Display_Local_Library:R_Custom R?
 U 1 1 5BC42848
 P 8000 4980
@@
 $EndComp
 $Comp
-L Custom_Library:R_Custom R?
+L LED_Display_Local_Library:R_Custom R?
 U 1 1 5BC42859
 P 7240 4680
@@
 F 2 "Resistors_SMD:R_0603" H 7240 4680 50  0001 C CNN
 F 3 "" H 7240 4680 50  0001 C CNN
-F 4 "0603" H 7320 4760 50  0000 L CNN "display_footprint"
-F 5 "1%" H 7320 4680 50  0000 L CNN "Tolerance"
-F 6 "1/10W" H 7320 4600 50  0000 L CNN "Wattage"
-F 7 "RHM10KADCT-ND" H 7540 5080 60  0001 C CNN "Digi-Key PN"
+F 4 "RHM10KADCT-ND" H 7540 5080 60  0001 C CNN "Digi-Key PN"
+F 5 "0603" H 7320 4760 50  0000 L CNN "display_footprint"
+F 6 "1%" H 7320 4680 50  0000 L CNN "Tolerance"
+F 7 "1/10W" H 7320 4600 50  0000 L CNN "Wattage"
 	1    7240 4680
 	1    0    0    -1
@@
 	7240 4460 7700 4460
 $Comp
-L Custom_Library:R_Custom R1104
+L LED_Display_Local_Library:R_Custom R1104
 U 1 1 5BC4286C
 P 6560 4460
@@
 F 2 "Resistors_SMD:R_0603" H 6560 4460 50  0001 C CNN
 F 3 "" H 6560 4460 50  0001 C CNN
-F 4 "0603" V 6660 4460 50  0000 C CNN "display_footprint"
-F 5 "1%" V 6760 4460 50  0000 C CNN "Tolerance"
-F 6 "1/10W" V 6860 4460 50  0000 C CNN "Wattage"
-F 7 "YAG3351CT-ND" H 6860 4860 60  0001 C CNN "Digi-Key PN"
+F 4 "YAG3351CT-ND" H 6860 4860 60  0001 C CNN "Digi-Key PN"
+F 5 "0603" V 6660 4460 50  0000 C CNN "display_footprint"
+F 6 "1%" V 6760 4460 50  0000 C CNN "Tolerance"
+F 7 "1/10W" V 6860 4460 50  0000 C CNN "Wattage"
 	1    6560 4460
 	0    1    1    0
@@
 LOAD_GATE
 $Comp
-L Custom_Library:C_Custom C?
+L LED_Display_Local_Library:C_Custom C?
 U 1 1 5BC368AD
 P 2640 4780
@@
 F 2 "Capacitors_SMD:C_0603" H 2678 4630 50  0001 C CNN
 F 3 "" H 2665 4880 50  0001 C CNN
-F 4 "0603" H 2490 4880 50  0000 R CNN "display_footprint"
-F 5 "16V" H 2490 4780 50  0000 R CNN "Voltage"
-F 6 "X7R" H 2490 4680 50  0000 R CNN "Dielectric"
-F 7 "1276-6524-1-ND" H 3065 5280 60  0001 C CNN "Digi-Key PN"
+F 4 "1276-6524-1-ND" H 3065 5280 60  0001 C CNN "Digi-Key PN"
+F 5 "0603" H 2490 4880 50  0000 R CNN "display_footprint"
+F 6 "16V" H 2490 4780 50  0000 R CNN "Voltage"
+F 7 "X7R" H 2490 4680 50  0000 R CNN "Dielectric"
 	1    2640 4780
 	1    0    0    -1
@@
 $EndComp
 $Comp
-L Custom_Library:C_Custom C?
+L LED_Display_Local_Library:C_Custom C?
 U 1 1 5BC368C8
 P 3310 4780
@@
 F 2 "Capacitors_SMD:C_0603" H 3348 4630 50  0001 C CNN
 F 3 "" H 3335 4880 50  0001 C CNN
-F 4 "0603" H 3160 4880 50  0000 R CNN "display_footprint"
-F 5 "50V" H 3160 4780 50  0000 R CNN "Voltage"
-F 6 "X7R" H 3160 4680 50  0000 R CNN "Dielectric"
-F 7 "490-4779-1-ND" H 3735 5280 60  0001 C CNN "Digi-Key PN"
+F 4 "490-4779-1-ND" H 3735 5280 60  0001 C CNN "Digi-Key PN"
+F 5 "0603" H 3160 4880 50  0000 R CNN "display_footprint"
+F 6 "50V" H 3160 4780 50  0000 R CNN "Voltage"
+F 7 "X7R" H 3160 4680 50  0000 R CNN "Dielectric"
 	1    3310 4780
 	1    0    0    -1
@@
 $EndComp
 $Comp
-L Custom_Library:CP_Tant_Custom C?
+L LED_Display_Local_Library:CP_Tant_Custom C?
 U 1 1 5BC376D5
 P 3920 4780
@@
 $EndComp
 Text Notes 540  690  0    100  ~ 20
-Active Load Driver and Active Load Bank 1
+11. Active Load Driver and Active Load Bank 1
 Wire Wire Line
 	8000 4660 8000 4830
+$Comp
+L LED_Display_Local_Library:MU_Logo #G?
+U 1 1 5C003EF4
+P 9900 1100
+F 0 "#G?" H 9900 614 60  0001 C CNN
+F 1 "MU_Logo" H 9900 1586 60  0001 C CNN
+F 2 "" H 9900 1100 50  0001 C CNN
+F 3 "" H 9900 1100 50  0001 C CNN
+	1    9900 1100
+	1    0    0    -1
+$EndComp
 $EndSCHEMATC

Commit message: Schematic cleanup
Other:
- moved on the sheet: C1103
Changed lines of the file:
@@
 Date "2018-11-28"
 Rev "A"
-Comp "Marquette Senior Design 2018, Group E44"
+Comp "Marquette University Senior Design 2018 Group E44"
 Comment1 ""
 Comment2 ""
@@
 U 1 1 5BC35FFA
 P 8830 2700
-F 0 "J1102" H 8830 2800 50  0000 C CNN
-F 1 "ISNS" H 8830 2500 50  0000 C CNN
+F 0 "J1102" H 8910 2692 50  0000 L CNN
+F 1 "ISNS" H 8910 2601 50  0000 L CNN
 F 2 "Pin_Headers:Pin_Header_Straight_1x02_Pitch2.54mm" H 8830 2700 50  0001 C CNN
 F 3 "~" H 8830 2700 50  0001 C CNN
@@
 AR Path="/5BB86F29/5BC370E8" Ref="R?"  Part="1"
 AR Path="/5BBF20D5/5BC370E8" Ref="R1107"  Part="1"
-F 0 "R1107" H 7900 2940 50  0000 R CNN
+F 0 "R1107" H 7940 2940 50  0000 R CNN
 F 1 "5m" V 8000 2940 50  0000 C CNN
 F 2 "Resistors_SMD:R_2512" H 8000 2940 50  0001 C CNN
@@
 AR Path="/5BB86F23/5BC37C2E" Ref="R?"  Part="1"
 AR Path="/5BBF20D5/5BC37C2E" Ref="R1105"  Part="1"
-F 0 "R1105" H 7140 2640 50  0000 R CNN
+F 0 "R1105" H 7180 2640 50  0000 R CNN
 F 1 "10k" V 7240 2640 50  0000 C CNN
 F 2 "Resistors_SMD:R_0603" H 7240 2640 50  0001 C CNN
@@
 U 1 1 5BC411E6
 P 1670 3510
-F 0 "J1101" H 1670 3610 50  0000 C CNN
-F 1 "FG_LOAD" H 1670 3310 50  0000 C CNN
+F 0 "J1101" H 1750 3520 50  0000 L CNN
+F 1 "FG_LOAD" H 1750 3440 50  0000 L CNN
 F 2 "Pin_Headers:Pin_Header_Straight_1x02_Pitch2.54mm" H 1670 3510 50  0001 C CNN
 F 3 "~" H 1670 3510 50  0001 C CNN
@@
 AR Path="/5BB86F23/5BC41AD3" Ref="R?"  Part="1"
 AR Path="/5BBF20D5/5BC41AD3" Ref="R1101"  Part="1"
-F 0 "R1101" H 2400 3730 50  0000 R CNN
+F 0 "R1101" H 2440 3730 50  0000 R CNN
 F 1 "10k" V 2500 3730 50  0000 C CNN
 F 2 "Resistors_SMD:R_0603" H 2500 3730 50  0001 C CNN
@@
 AR Path="/5BB86F29/5BC42848" Ref="R?"  Part="1"
 AR Path="/5BBF20D5/5BC42848" Ref="R1108"  Part="1"
-F 0 "R1108" H 7900 4980 50  0000 R CNN
+F 0 "R1108" H 7940 4980 50  0000 R CNN
 F 1 "5m" V 8000 4980 50  0000 C CNN
 F 2 "Resistors_SMD:R_2512" H 8000 4980 50  0001 C CNN
@@
 AR Path="/5BB86F23/5BC42859" Ref="R?"  Part="1"
 AR Path="/5BBF20D5/5BC42859" Ref="R1106"  Part="1"
-F 0 "R1106" H 7140 4680 50  0000 R CNN
+F 0 "R1106" H 7180 4680 50  0000 R CNN
 F 1 "10k" V 7240 4680 50  0000 C CNN
 F 2 "Resistors_SMD:R_0603" H 7240 4680 50  0001 C CNN
@@
 L LED_Display_Local_Library:CP_Tant_Custom C?
 U 1 1 5BC376D5
-P 3920 4780
+P 3980 4780
 AR Path="/5BB86F29/5BC376D5" Ref="C?"  Part="1"
 AR Path="/5BB86F2C/5BC376D5" Ref="C?"  Part="1"
@@
 AR Path="/5BB9CE4B/5BC376D5" Ref="C?"  Part="1"
 AR Path="/5BBF20D5/5BC376D5" Ref="C1103"  Part="1"
-F 0 "C1103" H 3945 4880 50  0000 L CNN
-F 1 "10uF" H 3945 4680 50  0000 L CNN
-F 2 "Capacitors_Tantalum_SMD:CP_Tantalum_Case-B_EIA-3528-21_Reflow" H 3958 4630 50  0001 C CNN
-F 3 "" H 3945 4880 50  0001 C CNN
-F 4 "399-5034-1-ND" H 3920 4780 50  0001 C CNN "Digi-Key PN"
-F 5 "3528" H 3770 4880 50  0000 R CNN "display_footprint"
-F 6 "16V" H 3770 4780 50  0000 R CNN "Voltage"
-F 7 "10%" H 3770 4680 50  0000 R CNN "Tolerance"
-	1    3920 4780
+F 0 "C1103" H 4005 4880 50  0000 L CNN
+F 1 "10uF" H 4005 4680 50  0000 L CNN
+F 2 "Capacitors_Tantalum_SMD:CP_Tantalum_Case-B_EIA-3528-21_Reflow" H 4018 4630 50  0001 C CNN
+F 3 "" H 4005 4880 50  0001 C CNN
+F 4 "399-5034-1-ND" H 3980 4780 50  0001 C CNN "Digi-Key PN"
+F 5 "3528" H 3830 4880 50  0000 R CNN "display_footprint"
+F 6 "16V" H 3830 4780 50  0000 R CNN "Voltage"
+F 7 "10%" H 3830 4680 50  0000 R CNN "Tolerance"
+	1    3980 4780
 	1    0    0    -1
 $EndComp
@@
 L power:+12V #PWR01110
 U 1 1 5BC37868
-P 3920 4630
-F 0 "#PWR01110" H 3920 4480 50  0001 C CNN
-F 1 "+12V" H 3920 4770 50  0000 C CNN
-F 2 "" H 3920 4630 50  0001 C CNN
-F 3 "" H 3920 4630 50  0001 C CNN
-	1    3920 4630
+P 3980 4630
+F 0 "#PWR01110" H 3980 4480 50  0001 C CNN
+F 1 "+12V" H 3980 4770 50  0000 C CNN
+F 2 "" H 3980 4630 50  0001 C CNN
+F 3 "" H 3980 4630 50  0001 C CNN
+	1    3980 4630
 	1    0    0    -1
 $EndComp
@@
 L power:GND #PWR?
 U 1 1 5BC37895
-P 3920 4930
+P 3980 4930
 AR Path="/5BB86F29/5BC37895" Ref="#PWR?"  Part="1"
 AR Path="/5BBF20D5/5BC37895" Ref="#PWR01111"  Part="1"
-F 0 "#PWR01111" H 3920 4680 50  0001 C CNN
-F 1 "GND" H 3920 4780 50  0000 C CNN
-F 2 "" H 3920 4930 50  0001 C CNN
-F 3 "" H 3920 4930 50  0001 C CNN
-	1    3920 4930
-	1    0    0    -1
-$EndComp
+F 0 "#PWR01111" H 3980 4680 50  0001 C CNN
+F 1 "GND" H 3980 4780 50  0000 C CNN
+F 2 "" H 3980 4930 50  0001 C CNN
+F 3 "" H 3980 4930 50  0001 C CNN
+	1    3980 4930
+	1    0    0    -1
+$EndComp
