File: hdw/Power_Board/LTC7851_Demo/Active_Load_3.sch (KiCad schematic (older format))
At the start: 8 parts, among them Q1301 IPC100N04S51R7ATMA1, Q1302 IPC100N04S51R7ATMA1

Commit message: Merging drews_branch_3 into master
Parts:
- R1301, R1302, R1303, R1304, R1305, R1306: symbol Custom_Library:R_Custom -> LED_Display_Local_Library:R_Custom
Other:
- note added: "13. Active Load Bank 3"
- note removed: "Active Load Bank 3"
Changed lines of the file:
@@
 $EndComp
 $Comp
-L Custom_Library:R_Custom R?
+L LED_Display_Local_Library:R_Custom R?
 U 1 1 5BC437F8
 P 8000 2940
@@
 $EndComp
 $Comp
-L Custom_Library:R_Custom R?
+L LED_Display_Local_Library:R_Custom R?
 U 1 1 5BC43809
 P 7240 2640
@@
 F 2 "Resistors_SMD:R_0603" H 7240 2640 50  0001 C CNN
 F 3 "" H 7240 2640 50  0001 C CNN
-F 4 "0603" H 7320 2720 50  0000 L CNN "display_footprint"
-F 5 "1%" H 7320 2640 50  0000 L CNN "Tolerance"
-F 6 "1/10W" H 7320 2560 50  0000 L CNN "Wattage"
-F 7 "RHM10KADCT-ND" H 7540 3040 60  0001 C CNN "Digi-Key PN"
+F 4 "RHM10KADCT-ND" H 7540 3040 60  0001 C CNN "Digi-Key PN"
+F 5 "0603" H 7320 2720 50  0000 L CNN "display_footprint"
+F 6 "1%" H 7320 2640 50  0000 L CNN "Tolerance"
+F 7 "1/10W" H 7320 2560 50  0000 L CNN "Wattage"
 	1    7240 2640
 	1    0    0    -1
@@
 	7240 2420 7700 2420
 $Comp
-L Custom_Library:R_Custom R1301
+L LED_Display_Local_Library:R_Custom R1301
 U 1 1 5BC4381C
 P 6560 2420
@@
 F 2 "Resistors_SMD:R_0603" H 6560 2420 50  0001 C CNN
 F 3 "" H 6560 2420 50  0001 C CNN
-F 4 "0603" V 6660 2420 50  0000 C CNN "display_footprint"
-F 5 "1%" V 6760 2420 50  0000 C CNN "Tolerance"
-F 6 "1/10W" V 6860 2420 50  0000 C CNN "Wattage"
-F 7 "YAG3351CT-ND" H 6860 2820 60  0001 C CNN "Digi-Key PN"
+F 4 "YAG3351CT-ND" H 6860 2820 60  0001 C CNN "Digi-Key PN"
+F 5 "0603" V 6660 2420 50  0000 C CNN "display_footprint"
+F 6 "1%" V 6760 2420 50  0000 C CNN "Tolerance"
+F 7 "1/10W" V 6860 2420 50  0000 C CNN "Wattage"
 	1    6560 2420
 	0    1    1    0
@@
 $EndComp
 $Comp
-L Custom_Library:R_Custom R?
+L LED_Display_Local_Library:R_Custom R?
 U 1 1 5BC43849
 P 8000 4980
@@
 $EndComp
 $Comp
-L Custom_Library:R_Custom R?
+L LED_Display_Local_Library:R_Custom R?
 U 1 1 5BC4385A
 P 7240 4680
@@
 F 2 "Resistors_SMD:R_0603" H 7240 4680 50  0001 C CNN
 F 3 "" H 7240 4680 50  0001 C CNN
-F 4 "0603" H 7320 4760 50  0000 L CNN "display_footprint"
-F 5 "1%" H 7320 4680 50  0000 L CNN "Tolerance"
-F 6 "1/10W" H 7320 4600 50  0000 L CNN "Wattage"
-F 7 "RHM10KADCT-ND" H 7540 5080 60  0001 C CNN "Digi-Key PN"
+F 4 "RHM10KADCT-ND" H 7540 5080 60  0001 C CNN "Digi-Key PN"
+F 5 "0603" H 7320 4760 50  0000 L CNN "display_footprint"
+F 6 "1%" H 7320 4680 50  0000 L CNN "Tolerance"
+F 7 "1/10W" H 7320 4600 50  0000 L CNN "Wattage"
 	1    7240 4680
 	1    0    0    -1
@@
 	7240 4460 7700 4460
 $Comp
-L Custom_Library:R_Custom R1302
+L LED_Display_Local_Library:R_Custom R1302
 U 1 1 5BC4386D
 P 6560 4460
@@
 F 2 "Resistors_SMD:R_0603" H 6560 4460 50  0001 C CNN
 F 3 "" H 6560 4460 50  0001 C CNN
-F 4 "0603" V 6660 4460 50  0000 C CNN "display_footprint"
-F 5 "1%" V 6760 4460 50  0000 C CNN "Tolerance"
-F 6 "1/10W" V 6860 4460 50  0000 C CNN "Wattage"
-F 7 "YAG3351CT-ND" H 6860 4860 60  0001 C CNN "Digi-Key PN"
+F 4 "YAG3351CT-ND" H 6860 4860 60  0001 C CNN "Digi-Key PN"
+F 5 "0603" V 6660 4460 50  0000 C CNN "display_footprint"
+F 6 "1%" V 6760 4460 50  0000 C CNN "Tolerance"
+F 7 "1/10W" V 6860 4460 50  0000 C CNN "Wattage"
 	1    6560 4460
 	0    1    1    0
@@
 LOAD_GATE
 Text Notes 540  690  0    100  ~ 20
-Active Load Bank 3
+13. Active Load Bank 3
 Wire Wire Line
 	8000 2620 8000 2790
 Wire Wire Line
 	8000 4660 8000 4830
+$Comp
+L LED_Display_Local_Library:MU_Logo #G?
+U 1 1 5C003F88
+P 9900 1100
+F 0 "#G?" H 9900 614 60  0001 C CNN
+F 1 "MU_Logo" H 9900 1586 60  0001 C CNN
+F 2 "" H 9900 1100 50  0001 C CNN
+F 3 "" H 9900 1100 50  0001 C CNN
+	1    9900 1100
+	1    0    0    -1
+$EndComp
 $EndSCHEMATC

Commit message: Schematic cleanup
Changed lines of the file:
@@
 Date "2018-11-28"
 Rev "A"
-Comp "Marquette Senior Design 2018, Group E44"
+Comp "Marquette University Senior Design 2018 Group E44"
 Comment1 ""
 Comment2 ""
@@
 AR Path="/5BBF20D5/5BC437F8" Ref="R?"  Part="1"
 AR Path="/5BBF20DB/5BC437F8" Ref="R1305"  Part="1"
-F 0 "R1305" H 7900 2940 50  0000 R CNN
+F 0 "R1305" H 7940 2940 50  0000 R CNN
 F 1 "5m" V 8000 2940 50  0000 C CNN
 F 2 "Resistors_SMD:R_2512" H 8000 2940 50  0001 C CNN
@@
 AR Path="/5BBF20D5/5BC43809" Ref="R?"  Part="1"
 AR Path="/5BBF20DB/5BC43809" Ref="R1303"  Part="1"
-F 0 "R1303" H 7140 2640 50  0000 R CNN
+F 0 "R1303" H 7180 2640 50  0000 R CNN
 F 1 "10k" V 7240 2640 50  0000 C CNN
 F 2 "Resistors_SMD:R_0603" H 7240 2640 50  0001 C CNN
@@
 AR Path="/5BBF20D5/5BC43849" Ref="R?"  Part="1"
 AR Path="/5BBF20DB/5BC43849" Ref="R1306"  Part="1"
-F 0 "R1306" H 7900 4980 50  0000 R CNN
+F 0 "R1306" H 7940 4980 50  0000 R CNN
 F 1 "5m" V 8000 4980 50  0000 C CNN
 F 2 "Resistors_SMD:R_2512" H 8000 4980 50  0001 C CNN
@@
 AR Path="/5BBF20D5/5BC4385A" Ref="R?"  Part="1"
 AR Path="/5BBF20DB/5BC4385A" Ref="R1304"  Part="1"
-F 0 "R1304" H 7140 4680 50  0000 R CNN
+F 0 "R1304" H 7180 4680 50  0000 R CNN
 F 1 "10k" V 7240 4680 50  0000 C CNN
 F 2 "Resistors_SMD:R_0603" H 7240 4680 50  0001 C CNN
