File: hdw/Power_Board/LTC7851_Demo/Loop_Response.sch (KiCad schematic (older format))
At the start: 4 parts, among them J1401 VOUT, J1402 LOOP_TAP, J1403 Wave_Gen_In, T1401 1:1 Pulse Transformer

Commit message: Merging drews_branch_3 into master
Other:
- note added: "14. Open Loop Transfer Function Test Components"
- note removed: "Open Loop Transfer Function Test Components"
Changed lines of the file:
@@
 Connection ~ 5640 4050
 Text Notes 540  690  0    100  ~ 20
-Open Loop Transfer Function Test Components
+14. Open Loop Transfer Function Test Components
+$Comp
+L LED_Display_Local_Library:MU_Logo #G?
+U 1 1 5C003FC2
+P 9900 1100
+F 0 "#G?" H 9900 614 60  0001 C CNN
+F 1 "MU_Logo" H 9900 1586 60  0001 C CNN
+F 2 "" H 9900 1100 50  0001 C CNN
+F 3 "" H 9900 1100 50  0001 C CNN
+	1    9900 1100
+	1    0    0    -1
+$EndComp
 $EndSCHEMATC
