File: hdw/Power_Board/LTC7851_Demo/Power_Output.sch (KiCad schematic (older format))
At the start: 4 parts, among them J901 +5V OUT, J902 +5V OUT, J903 GND OUT, J904 GND OUT

Commit message: Merging drews_branch_3 into master
Other:
- note added: "09. Power Output"
- note removed: "Power Output"
Changed lines of the file:
@@
 Place bulk output caps close to terminals
 Text Notes 540  690  0    100  ~ 20
-Power Output
+09. Power Output
+$Comp
+L LED_Display_Local_Library:MU_Logo #G?
+U 1 1 5C003E58
+P 9900 1100
+F 0 "#G?" H 9900 614 60  0001 C CNN
+F 1 "MU_Logo" H 9900 1586 60  0001 C CNN
+F 2 "" H 9900 1100 50  0001 C CNN
+F 3 "" H 9900 1100 50  0001 C CNN
+	1    9900 1100
+	1    0    0    -1
+$EndComp
 $EndSCHEMATC
