File: hdw/Logic_Board/LED_Display_Controller/Power_Input.sch (KiCad schematic (older format))
At the start: 22 parts, among them J201 +12V IN, J202 GND IN, J203 +12V IN AUX, J204 Master Power SW, Q201 IPC100N04S51R7ATMA1, Q202 IPC100N04S51R7ATMA1, U201 LTC4365DDB

Commit message: Added some digikey partnumbers to components
Parts:
- C201, C204: Digi-Key PN 490-4779-1-ND -> 311-1344-1-ND
- C203: Digi-Key PN 311-1080-1-ND -> 1276-1018-1-ND
- R201: footprint Resistors_SMD:R_0603 -> (none); Digi-Key PN 541-6.04MHCT-ND -> PN
- R202: footprint Resistors_SMD:R_0603 -> (none); Digi-Key PN 311-86.6KHRCT-ND -> PN
- R203: footprint Resistors_SMD:R_0603 -> (none); Digi-Key PN 541-243KHCT-ND -> PN
- R204: footprint Resistors_SMD:R_0603 -> (none); Digi-Key PN P100KHCT-ND -> PN
- R205, R206: footprint Resistors_SMD:R_0603 -> (none); Digi-Key PN YAG3351CT-ND -> PN
- R207: footprint Resistors_SMD:R_0603 -> (none); Digi-Key PN RHM10KADCT-ND -> PN
- R208: footprint Resistors_SMD:R_0603 -> (none); Digi-Key PN RMCF0603FT5K10CT-ND -> PN
- U201: footprint Package_DFN_QFN:DFN-8-1EP_2x3mm_P0.5mm_EP0.61x2.2mm -> (none)
Changed lines of the file:
@@
 F 0 "R201" H 3290 4050 50  0000 R CNN
 F 1 "6.04M" V 3350 4050 40  0000 C CNN
-F 2 "Resistors_SMD:R_0603" H 3350 4050 50  0001 C CNN
+F 2 "" H 3350 4050 50  0001 C CNN
 F 3 "" H 3350 4050 50  0001 C CNN
-F 4 "541-6.04MHCT-ND" H 3650 4450 60  0001 C CNN "Digi-Key PN"
+F 4 "PN" H 3650 4450 60  0001 C CNN "Digi-Key PN"
 F 5 "0603" H 3430 4130 50  0000 L CNN "display_footprint"
 F 6 "1%" H 3430 4050 50  0000 L CNN "Tolerance"
@@
 F 5 "50V" H 5510 5790 50  0000 R CNN "Voltage"
 F 6 "X7R" H 5510 5690 50  0000 R CNN "Dielectric"
-F 7 "490-4779-1-ND" H 6085 6290 60  0001 C CNN "Digi-Key PN"
+F 7 "311-1344-1-ND" H 6085 6290 60  0001 C CNN "Digi-Key PN"
 	1    5660 5790
 	1    0    0    -1
@@
 F 5 "50V" H 6110 5790 50  0001 R CNN "Voltage"
 F 6 "X7R" H 6110 5690 50  0001 R CNN "Dielectric"
-F 7 "311-1080-1-ND" H 6685 6290 60  0001 C CNN "Digi-Key PN"
+F 7 "1276-1018-1-ND" H 6685 6290 60  0001 C CNN "Digi-Key PN"
 	1    6260 5790
 	1    0    0    -1
@@
 F 0 "R202" H 3290 4580 50  0000 R CNN
 F 1 "86.6k" V 3350 4580 40  0000 C CNN
-F 2 "Resistors_SMD:R_0603" H 3350 4580 50  0001 C CNN
+F 2 "" H 3350 4580 50  0001 C CNN
 F 3 "" H 3350 4580 50  0001 C CNN
-F 4 "311-86.6KHRCT-ND" H 3650 4980 60  0001 C CNN "Digi-Key PN"
+F 4 "PN" H 3650 4980 60  0001 C CNN "Digi-Key PN"
 F 5 "0603" H 3430 4660 50  0000 L CNN "display_footprint"
 F 6 "1%" H 3430 4580 50  0000 L CNN "Tolerance"
@@
 F 0 "R203" H 3290 5080 50  0000 R CNN
 F 1 "243k" V 3350 5080 40  0000 C CNN
-F 2 "Resistors_SMD:R_0603" H 3350 5080 50  0001 C CNN
+F 2 "" H 3350 5080 50  0001 C CNN
 F 3 "" H 3350 5080 50  0001 C CNN
-F 4 "541-243KHCT-ND" H 3650 5480 60  0001 C CNN "Digi-Key PN"
+F 4 "PN" H 3650 5480 60  0001 C CNN "Digi-Key PN"
 F 5 "0603" H 3430 5160 50  0000 L CNN "display_footprint"
 F 6 "1%" H 3430 5080 50  0000 L CNN "Tolerance"
@@
 F 0 "R204" H 3820 3560 50  0000 R CNN
 F 1 "100k" V 3880 3560 40  0000 C CNN
-F 2 "Resistors_SMD:R_0603" H 3880 3560 50  0001 C CNN
+F 2 "" H 3880 3560 50  0001 C CNN
 F 3 "" H 3880 3560 50  0001 C CNN
-F 4 "P100KHCT-ND" H 4180 3960 60  0001 C CNN "Digi-Key PN"
+F 4 "PN" H 4180 3960 60  0001 C CNN "Digi-Key PN"
 F 5 "0603" H 3960 3640 50  0000 L CNN "display_footprint"
 F 6 "1%" H 3960 3560 50  0000 L CNN "Tolerance"
@@
 F 0 "R205" V 5330 2630 50  0000 C CNN
 F 1 "10" V 5430 2630 50  0000 C CNN
-F 2 "Resistors_SMD:R_0603" H 5430 2630 50  0001 C CNN
+F 2 "" H 5430 2630 50  0001 C CNN
 F 3 "" H 5430 2630 50  0001 C CNN
-F 4 "YAG3351CT-ND" H 5730 3030 60  0001 C CNN "Digi-Key PN"
+F 4 "PN" H 5730 3030 60  0001 C CNN "Digi-Key PN"
 F 5 "0603" V 5530 2630 50  0000 C CNN "display_footprint"
 F 6 "1%" V 5630 2630 50  0000 C CNN "Tolerance"
@@
 F 0 "R206" V 6200 2630 50  0000 C CNN
 F 1 "10" V 6300 2630 50  0000 C CNN
-F 2 "Resistors_SMD:R_0603" H 6300 2630 50  0001 C CNN
+F 2 "" H 6300 2630 50  0001 C CNN
 F 3 "" H 6300 2630 50  0001 C CNN
-F 4 "YAG3351CT-ND" H 6600 3030 60  0001 C CNN "Digi-Key PN"
+F 4 "PN" H 6600 3030 60  0001 C CNN "Digi-Key PN"
 F 5 "0603" V 6400 2630 50  0000 C CNN "display_footprint"
 F 6 "1%" V 6500 2630 50  0000 C CNN "Tolerance"
@@
 F 0 "R208" H 7450 3540 50  0000 R CNN
 F 1 "5.1k" V 7510 3540 50  0000 C CNN
-F 2 "Resistors_SMD:R_0603" H 7510 3540 50  0001 C CNN
+F 2 "" H 7510 3540 50  0001 C CNN
 F 3 "" H 7510 3540 50  0001 C CNN
-F 4 "RMCF0603FT5K10CT-ND" H 7810 3940 60  0001 C CNN "Digi-Key PN"
+F 4 "PN" H 7810 3940 60  0001 C CNN "Digi-Key PN"
 F 5 "0603" H 7590 3620 50  0000 L CNN "display_footprint"
 F 6 "1%" H 7590 3540 50  0000 L CNN "Tolerance"
@@
 F 0 "R207" H 6500 3930 50  0000 R CNN
 F 1 "10k" V 6560 3930 50  0000 C CNN
-F 2 "Resistors_SMD:R_0603" H 6560 3930 50  0001 C CNN
+F 2 "" H 6560 3930 50  0001 C CNN
 F 3 "" H 6560 3930 50  0001 C CNN
-F 4 "RHM10KADCT-ND" H 6860 4330 60  0001 C CNN "Digi-Key PN"
+F 4 "PN" H 6860 4330 60  0001 C CNN "Digi-Key PN"
 F 5 "0603" H 6640 4010 50  0000 L CNN "display_footprint"
 F 6 "1%" H 6640 3930 50  0000 L CNN "Tolerance"
@@
 F 0 "U201" H 5570 4960 50  0000 L CNN
 F 1 "LTC4365DDB" H 5920 4960 50  0000 L CNN
-F 2 "Package_DFN_QFN:DFN-8-1EP_2x3mm_P0.5mm_EP0.61x2.2mm" H 5870 4060 50  0001 C CNN
+F 2 "" H 5870 4060 50  0001 C CNN
 F 3 "http://cds.linear.com/docs/en/datasheet/4365fa.pdf" H 5870 4310 50  0001 C CNN
 F 4 "LTC4365IDDB#TRMPBFCT-ND" H 5870 4060 50  0001 C CNN "Digi-Key PN"
@@
 F 5 "50V" H 7360 3840 50  0000 R CNN "Voltage"
 F 6 "X7R" H 7360 3740 50  0000 R CNN "Dielectric"
-F 7 "490-4779-1-ND" H 7935 4340 60  0001 C CNN "Digi-Key PN"
+F 7 "311-1344-1-ND" H 7935 4340 60  0001 C CNN "Digi-Key PN"
 	1    7510 3840
 	1    0    0    -1

Commit message: Finished first pass of digikey part numbers
Parts:
- J203: Digi-Key PN (none) -> CP-202BH-ND
- R201: Digi-Key PN PN -> 541-6.04MHCT-ND
- R202: Digi-Key PN PN -> 311-86.6KHRCT-ND
- R203: Digi-Key PN PN -> 311-243KHRCT-ND
- R204: Digi-Key PN PN -> A106046CT-ND
- R205, R206: Digi-Key PN PN -> YAG3351CT-ND
- R207: Digi-Key PN PN -> RMCF0603FT10K0CT-ND
- R208: Digi-Key PN PN -> YAG3621CT-ND
Changed lines of the file:
@@
 F 2 "" H 3350 4050 50  0001 C CNN
 F 3 "" H 3350 4050 50  0001 C CNN
-F 4 "PN" H 3650 4450 60  0001 C CNN "Digi-Key PN"
+F 4 "541-6.04MHCT-ND" H 3650 4450 60  0001 C CNN "Digi-Key PN"
 F 5 "0603" H 3430 4130 50  0000 L CNN "display_footprint"
 F 6 "1%" H 3430 4050 50  0000 L CNN "Tolerance"
@@
 F 2 "" H 3350 4580 50  0001 C CNN
 F 3 "" H 3350 4580 50  0001 C CNN
-F 4 "PN" H 3650 4980 60  0001 C CNN "Digi-Key PN"
+F 4 "311-86.6KHRCT-ND" H 3650 4980 60  0001 C CNN "Digi-Key PN"
 F 5 "0603" H 3430 4660 50  0000 L CNN "display_footprint"
 F 6 "1%" H 3430 4580 50  0000 L CNN "Tolerance"
@@
 F 2 "" H 3350 5080 50  0001 C CNN
 F 3 "" H 3350 5080 50  0001 C CNN
-F 4 "PN" H 3650 5480 60  0001 C CNN "Digi-Key PN"
+F 4 "311-243KHRCT-ND" H 3650 5480 60  0001 C CNN "Digi-Key PN"
 F 5 "0603" H 3430 5160 50  0000 L CNN "display_footprint"
 F 6 "1%" H 3430 5080 50  0000 L CNN "Tolerance"
@@
 F 2 "" H 3880 3560 50  0001 C CNN
 F 3 "" H 3880 3560 50  0001 C CNN
-F 4 "PN" H 4180 3960 60  0001 C CNN "Digi-Key PN"
+F 4 "A106046CT-ND" H 4180 3960 60  0001 C CNN "Digi-Key PN"
 F 5 "0603" H 3960 3640 50  0000 L CNN "display_footprint"
 F 6 "1%" H 3960 3560 50  0000 L CNN "Tolerance"
@@
 F 2 "" H 5430 2630 50  0001 C CNN
 F 3 "" H 5430 2630 50  0001 C CNN
-F 4 "PN" H 5730 3030 60  0001 C CNN "Digi-Key PN"
+F 4 "YAG3351CT-ND" H 5730 3030 60  0001 C CNN "Digi-Key PN"
 F 5 "0603" V 5530 2630 50  0000 C CNN "display_footprint"
 F 6 "1%" V 5630 2630 50  0000 C CNN "Tolerance"
@@
 F 2 "" H 6300 2630 50  0001 C CNN
 F 3 "" H 6300 2630 50  0001 C CNN
-F 4 "PN" H 6600 3030 60  0001 C CNN "Digi-Key PN"
+F 4 "YAG3351CT-ND" H 6600 3030 60  0001 C CNN "Digi-Key PN"
 F 5 "0603" V 6400 2630 50  0000 C CNN "display_footprint"
 F 6 "1%" V 6500 2630 50  0000 C CNN "Tolerance"
@@
 F 2 "" H 7510 3540 50  0001 C CNN
 F 3 "" H 7510 3540 50  0001 C CNN
-F 4 "PN" H 7810 3940 60  0001 C CNN "Digi-Key PN"
+F 4 "YAG3621CT-ND" H 7810 3940 60  0001 C CNN "Digi-Key PN"
 F 5 "0603" H 7590 3620 50  0000 L CNN "display_footprint"
 F 6 "1%" H 7590 3540 50  0000 L CNN "Tolerance"
@@
 F 2 "" H 6560 3930 50  0001 C CNN
 F 3 "" H 6560 3930 50  0001 C CNN
-F 4 "PN" H 6860 4330 60  0001 C CNN "Digi-Key PN"
+F 4 "RMCF0603FT10K0CT-ND" H 6860 4330 60  0001 C CNN "Digi-Key PN"
 F 5 "0603" H 6640 4010 50  0000 L CNN "display_footprint"
 F 6 "1%" H 6640 3930 50  0000 L CNN "Tolerance"
@@
 F 2 "" H 2210 2990 50  0001 C CNN
 F 3 "~" H 2210 2990 50  0001 C CNN
+F 4 "CP-202BH-ND" H 0   0   50  0001 C CNN "Digi-Key PN"
 	1    2160 3030
 	1    0    0    -1

Commit message: First pass assignment of footprints to all components
Parts:
- J201, J202: footprint (none) -> Electronic_Display_Footprint_Lib:Wuerth_7461096_M4_Shank_9pos
- J203: footprint (none) -> Connectors:BARREL_JACK
- J204: footprint (none) -> Pin_Headers:Pin_Header_Straight_1x02_Pitch2.54mm
- R201, R202, R203, R204, R205, R206, R207, R208: footprint (none) -> Resistors_SMD:R_0603
- U201: footprint (none) -> Housings_DFN_QFN:DFN-8-1EP_2x3mm_Pitch0.5mm
Changed lines of the file:
@@
 F 0 "R201" H 3290 4050 50  0000 R CNN
 F 1 "6.04M" V 3350 4050 40  0000 C CNN
-F 2 "" H 3350 4050 50  0001 C CNN
+F 2 "Resistors_SMD:R_0603" H 3350 4050 50  0001 C CNN
 F 3 "" H 3350 4050 50  0001 C CNN
 F 4 "541-6.04MHCT-ND" H 3650 4450 60  0001 C CNN "Digi-Key PN"
@@
 F 0 "R202" H 3290 4580 50  0000 R CNN
 F 1 "86.6k" V 3350 4580 40  0000 C CNN
-F 2 "" H 3350 4580 50  0001 C CNN
+F 2 "Resistors_SMD:R_0603" H 3350 4580 50  0001 C CNN
 F 3 "" H 3350 4580 50  0001 C CNN
 F 4 "311-86.6KHRCT-ND" H 3650 4980 60  0001 C CNN "Digi-Key PN"
@@
 F 0 "R203" H 3290 5080 50  0000 R CNN
 F 1 "243k" V 3350 5080 40  0000 C CNN
-F 2 "" H 3350 5080 50  0001 C CNN
+F 2 "Resistors_SMD:R_0603" H 3350 5080 50  0001 C CNN
 F 3 "" H 3350 5080 50  0001 C CNN
 F 4 "311-243KHRCT-ND" H 3650 5480 60  0001 C CNN "Digi-Key PN"
@@
 F 0 "R204" H 3820 3560 50  0000 R CNN
 F 1 "100k" V 3880 3560 40  0000 C CNN
-F 2 "" H 3880 3560 50  0001 C CNN
+F 2 "Resistors_SMD:R_0603" H 3880 3560 50  0001 C CNN
 F 3 "" H 3880 3560 50  0001 C CNN
 F 4 "A106046CT-ND" H 4180 3960 60  0001 C CNN "Digi-Key PN"
@@
 F 0 "R205" V 5330 2630 50  0000 C CNN
 F 1 "10" V 5430 2630 50  0000 C CNN
-F 2 "" H 5430 2630 50  0001 C CNN
+F 2 "Resistors_SMD:R_0603" H 5430 2630 50  0001 C CNN
 F 3 "" H 5430 2630 50  0001 C CNN
 F 4 "YAG3351CT-ND" H 5730 3030 60  0001 C CNN "Digi-Key PN"
@@
 F 0 "R206" V 6200 2630 50  0000 C CNN
 F 1 "10" V 6300 2630 50  0000 C CNN
-F 2 "" H 6300 2630 50  0001 C CNN
+F 2 "Resistors_SMD:R_0603" H 6300 2630 50  0001 C CNN
 F 3 "" H 6300 2630 50  0001 C CNN
 F 4 "YAG3351CT-ND" H 6600 3030 60  0001 C CNN "Digi-Key PN"
@@
 F 0 "R208" H 7450 3540 50  0000 R CNN
 F 1 "5.1k" V 7510 3540 50  0000 C CNN
-F 2 "" H 7510 3540 50  0001 C CNN
+F 2 "Resistors_SMD:R_0603" H 7510 3540 50  0001 C CNN
 F 3 "" H 7510 3540 50  0001 C CNN
 F 4 "YAG3621CT-ND" H 7810 3940 60  0001 C CNN "Digi-Key PN"
@@
 F 0 "R207" H 6500 3930 50  0000 R CNN
 F 1 "10k" V 6560 3930 50  0000 C CNN
-F 2 "" H 6560 3930 50  0001 C CNN
+F 2 "Resistors_SMD:R_0603" H 6560 3930 50  0001 C CNN
 F 3 "" H 6560 3930 50  0001 C CNN
 F 4 "RMCF0603FT10K0CT-ND" H 6860 4330 60  0001 C CNN "Digi-Key PN"
@@
 F 0 "J201" H 2110 2340 50  0000 C CNN
 F 1 "+12V IN" H 2110 2140 50  0000 C CNN
-F 2 "" H 2110 2240 50  0001 C CNN
+F 2 "Electronic_Display_Footprint_Lib:Wuerth_7461096_M4_Shank_9pos" H 2110 2240 50  0001 C CNN
 F 3 "~" H 2110 2240 50  0001 C CNN
 F 4 "732-3214-ND" H -3410 -410 50  0001 C CNN "Digi-Key PN"
@@
 F 0 "U201" H 5570 4960 50  0000 L CNN
 F 1 "LTC4365DDB" H 5920 4960 50  0000 L CNN
-F 2 "" H 5870 4060 50  0001 C CNN
+F 2 "Housings_DFN_QFN:DFN-8-1EP_2x3mm_Pitch0.5mm" H 5870 4060 50  0001 C CNN
 F 3 "http://cds.linear.com/docs/en/datasheet/4365fa.pdf" H 5870 4310 50  0001 C CNN
 F 4 "LTC4365IDDB#TRMPBFCT-ND" H 5870 4060 50  0001 C CNN "Digi-Key PN"
@@
 F 0 "J202" H 2110 4090 50  0000 C CNN
 F 1 "GND IN" H 2110 3890 50  0000 C CNN
-F 2 "" H 2110 3990 50  0001 C CNN
+F 2 "Electronic_Display_Footprint_Lib:Wuerth_7461096_M4_Shank_9pos" H 2110 3990 50  0001 C CNN
 F 3 "~" H 2110 3990 50  0001 C CNN
 F 4 "732-3214-ND" H -3410 1340 50  0001 C CNN "Digi-Key PN"
@@
 F 0 "J204" V 3884 6160 50  0000 L CNN
 F 1 "Master Power SW" V 3975 6160 50  0000 L CNN
-F 2 "" H 3880 6080 50  0001 C CNN
+F 2 "Pin_Headers:Pin_Header_Straight_1x02_Pitch2.54mm" H 3880 6080 50  0001 C CNN
 F 3 "~" H 3880 6080 50  0001 C CNN
 	1    3880 6080
@@
 F 0 "J203" H 2160 3240 50  0000 C CNN
 F 1 "+12V IN AUX" H 2160 2830 50  0000 C CNN
-F 2 "" H 2210 2990 50  0001 C CNN
+F 2 "Connectors:BARREL_JACK" H 2210 2990 50  0001 C CNN
 F 3 "~" H 2210 2990 50  0001 C CNN
 F 4 "CP-202BH-ND" H 0   0   50  0001 C CNN "Digi-Key PN"

Commit message: Resolved a few library dependencies
Parts:
- Q201, Q202: symbol Custom_Library:BSC032N04LSATMA1 -> LED_Display_Local_Library:IPC100N04S51R7ATMA1
Changed lines of the file:
@@
 Connection ~ 3880 3810
 $Comp
-L Custom_Library:BSC032N04LSATMA1 Q201
+L LED_Display_Local_Library:IPC100N04S51R7ATMA1 Q201
 U 1 1 5BED5FAB
 P 5200 2340
@@
 $EndComp
 $Comp
-L Custom_Library:BSC032N04LSATMA1 Q202
+L LED_Display_Local_Library:IPC100N04S51R7ATMA1 Q202
 U 1 1 5BEDD03C
 P 6550 2340
