File: hdw/Logic_Board/LED_Display_Controller/Status_LEDs_2.sch (KiCad schematic (older format))
At the start: 16 parts, among them U1301 74LVC1G06, U1302 74LVC1G06, U1303 74LVC1G06, U1304 74LVC1G06

Commit message: Added some digikey partnumbers to components
Parts:
- C1301, C1302, C1303, C1304: footprint (none) -> Capacitors_SMD:C_0603; Digi-Key PN PN -> 311-1344-1-ND
- D1301, D1302, D1303, D1304: Digi-Key PN (none) -> 160-1446-1-ND
Changed lines of the file:
@@
 F 0 "C1301" H 2295 4000 50  0000 L CNN
 F 1 "0.1uF" H 2295 3800 50  0000 L CNN
-F 2 "" H 2308 3750 50  0001 C CNN
+F 2 "Capacitors_SMD:C_0603" H 2308 3750 50  0001 C CNN
 F 3 "" H 2295 4000 50  0001 C CNN
-F 4 "PN" H 2695 4400 60  0001 C CNN "Digi-Key PN"
+F 4 "311-1344-1-ND" H 2695 4400 60  0001 C CNN "Digi-Key PN"
 F 5 "0603" H 2120 4000 50  0000 R CNN "display_footprint"
 F 6 "50V" H 2120 3900 50  0000 R CNN "Voltage"
@@
 F 0 "C1302" H 4645 4000 50  0000 L CNN
 F 1 "0.1uF" H 4645 3800 50  0000 L CNN
-F 2 "" H 4658 3750 50  0001 C CNN
+F 2 "Capacitors_SMD:C_0603" H 4658 3750 50  0001 C CNN
 F 3 "" H 4645 4000 50  0001 C CNN
-F 4 "PN" H 5045 4400 60  0001 C CNN "Digi-Key PN"
+F 4 "311-1344-1-ND" H 5045 4400 60  0001 C CNN "Digi-Key PN"
 F 5 "0603" H 4470 4000 50  0000 R CNN "display_footprint"
 F 6 "50V" H 4470 3900 50  0000 R CNN "Voltage"
@@
 F 0 "C1303" H 7025 4000 50  0000 L CNN
 F 1 "0.1uF" H 7025 3800 50  0000 L CNN
-F 2 "" H 7038 3750 50  0001 C CNN
+F 2 "Capacitors_SMD:C_0603" H 7038 3750 50  0001 C CNN
 F 3 "" H 7025 4000 50  0001 C CNN
-F 4 "PN" H 7425 4400 60  0001 C CNN "Digi-Key PN"
+F 4 "311-1344-1-ND" H 7425 4400 60  0001 C CNN "Digi-Key PN"
 F 5 "0603" H 6850 4000 50  0000 R CNN "display_footprint"
 F 6 "50V" H 6850 3900 50  0000 R CNN "Voltage"
@@
 F 0 "C1304" H 9275 4000 50  0000 L CNN
 F 1 "0.1uF" H 9275 3800 50  0000 L CNN
-F 2 "" H 9288 3750 50  0001 C CNN
+F 2 "Capacitors_SMD:C_0603" H 9288 3750 50  0001 C CNN
 F 3 "" H 9275 4000 50  0001 C CNN
-F 4 "PN" H 9675 4400 60  0001 C CNN "Digi-Key PN"
+F 4 "311-1344-1-ND" H 9675 4400 60  0001 C CNN "Digi-Key PN"
 F 5 "0603" H 9100 4000 50  0000 R CNN "display_footprint"
 F 6 "50V" H 9100 3900 50  0000 R CNN "Voltage"
@@
 F 2 "" H 2660 3000 50  0001 C CNN
 F 3 "~" H 2660 3000 50  0001 C CNN
+F 4 "160-1446-1-ND" H 0   0   50  0001 C CNN "Digi-Key PN"
 	1    2660 3000
 	0    -1   -1   0
@@
 F 2 "" H 5010 3000 50  0001 C CNN
 F 3 "~" H 5010 3000 50  0001 C CNN
+F 4 "160-1446-1-ND" H 0   0   50  0001 C CNN "Digi-Key PN"
 	1    5010 3000
 	0    -1   -1   0
@@
 F 2 "" H 7390 3000 50  0001 C CNN
 F 3 "~" H 7390 3000 50  0001 C CNN
+F 4 "160-1446-1-ND" H 0   0   50  0001 C CNN "Digi-Key PN"
 	1    7390 3000
 	0    -1   -1   0
@@
 F 2 "" H 9640 3000 50  0001 C CNN
 F 3 "~" H 9640 3000 50  0001 C CNN
+F 4 "160-1446-1-ND" H 0   0   50  0001 C CNN "Digi-Key PN"
 	1    9640 3000
 	0    -1   -1   0

Commit message: Finished first pass of digikey part numbers
Parts:
- R1301, R1302, R1303, R1304: Digi-Key PN PN -> RMCF0603FT1K00CT-ND
Changed lines of the file:
@@
 F 5 "1%" H 2730 2700 50  0000 L CNN "Tolerance"
 F 6 "1/10W" H 2730 2630 50  0000 L CNN "Wattage"
-F 7 "PN" H 2960 3100 60  0001 C CNN "Digi-Key PN"
+F 7 "RMCF0603FT1K00CT-ND" H 2960 3100 60  0001 C CNN "Digi-Key PN"
 	1    2660 2700
 	-1   0    0    -1
@@
 F 5 "1%" H 5080 2700 50  0000 L CNN "Tolerance"
 F 6 "1/10W" H 5080 2630 50  0000 L CNN "Wattage"
-F 7 "PN" H 5310 3100 60  0001 C CNN "Digi-Key PN"
+F 7 "RMCF0603FT1K00CT-ND" H 5310 3100 60  0001 C CNN "Digi-Key PN"
 	1    5010 2700
 	-1   0    0    -1
@@
 F 5 "1%" H 7460 2700 50  0000 L CNN "Tolerance"
 F 6 "1/10W" H 7460 2630 50  0000 L CNN "Wattage"
-F 7 "PN" H 7690 3100 60  0001 C CNN "Digi-Key PN"
+F 7 "RMCF0603FT1K00CT-ND" H 7690 3100 60  0001 C CNN "Digi-Key PN"
 	1    7390 2700
 	-1   0    0    -1
@@
 F 5 "1%" H 9710 2700 50  0000 L CNN "Tolerance"
 F 6 "1/10W" H 9710 2630 50  0000 L CNN "Wattage"
-F 7 "PN" H 9940 3100 60  0001 C CNN "Digi-Key PN"
+F 7 "RMCF0603FT1K00CT-ND" H 9940 3100 60  0001 C CNN "Digi-Key PN"
 	1    9640 2700
 	-1   0    0    -1

Commit message: First pass assignment of footprints to all components
Parts:
- D1301, D1302, D1303, D1304: footprint (none) -> LEDs:LED_0603
- R1301, R1302, R1303, R1304: footprint (none) -> Resistors_SMD:R_0603
Changed lines of the file:
@@
 F 0 "R1301" H 2600 2700 50  0000 R CNN
 F 1 "1k" V 2660 2700 50  0000 C CNN
-F 2 "" H 2660 2700 50  0001 C CNN
+F 2 "Resistors_SMD:R_0603" H 2660 2700 50  0001 C CNN
 F 3 "" H 2660 2700 50  0001 C CNN
 F 4 "0603" H 2730 2780 50  0000 L CNN "display_footprint"
@@
 F 0 "D1301" V 2698 2637 50  0000 L CNN
 F 1 "Green" V 2607 2883 50  0000 R CNN
-F 2 "" H 2660 3000 50  0001 C CNN
+F 2 "LEDs:LED_0603" H 2660 3000 50  0001 C CNN
 F 3 "~" H 2660 3000 50  0001 C CNN
 F 4 "160-1446-1-ND" H 0   0   50  0001 C CNN "Digi-Key PN"
@@
 F 0 "R1302" H 4950 2700 50  0000 R CNN
 F 1 "1k" V 5010 2700 50  0000 C CNN
-F 2 "" H 5010 2700 50  0001 C CNN
+F 2 "Resistors_SMD:R_0603" H 5010 2700 50  0001 C CNN
 F 3 "" H 5010 2700 50  0001 C CNN
 F 4 "0603" H 5080 2780 50  0000 L CNN "display_footprint"
@@
 F 0 "D1302" V 5048 2637 50  0000 L CNN
 F 1 "Green" V 4957 2883 50  0000 R CNN
-F 2 "" H 5010 3000 50  0001 C CNN
+F 2 "LEDs:LED_0603" H 5010 3000 50  0001 C CNN
 F 3 "~" H 5010 3000 50  0001 C CNN
 F 4 "160-1446-1-ND" H 0   0   50  0001 C CNN "Digi-Key PN"
@@
 F 0 "R1303" H 7330 2700 50  0000 R CNN
 F 1 "1k" V 7390 2700 50  0000 C CNN
-F 2 "" H 7390 2700 50  0001 C CNN
+F 2 "Resistors_SMD:R_0603" H 7390 2700 50  0001 C CNN
 F 3 "" H 7390 2700 50  0001 C CNN
 F 4 "0603" H 7460 2780 50  0000 L CNN "display_footprint"
@@
 F 0 "D1303" V 7428 2637 50  0000 L CNN
 F 1 "Green" V 7337 2883 50  0000 R CNN
-F 2 "" H 7390 3000 50  0001 C CNN
+F 2 "LEDs:LED_0603" H 7390 3000 50  0001 C CNN
 F 3 "~" H 7390 3000 50  0001 C CNN
 F 4 "160-1446-1-ND" H 0   0   50  0001 C CNN "Digi-Key PN"
@@
 F 0 "R1304" H 9580 2700 50  0000 R CNN
 F 1 "1k" V 9640 2700 50  0000 C CNN
-F 2 "" H 9640 2700 50  0001 C CNN
+F 2 "Resistors_SMD:R_0603" H 9640 2700 50  0001 C CNN
 F 3 "" H 9640 2700 50  0001 C CNN
 F 4 "0603" H 9710 2780 50  0000 L CNN "display_footprint"
@@
 F 0 "D1304" V 9678 2637 50  0000 L CNN
 F 1 "Green" V 9587 2883 50  0000 R CNN
-F 2 "" H 9640 3000 50  0001 C CNN
+F 2 "LEDs:LED_0603" H 9640 3000 50  0001 C CNN
 F 3 "~" H 9640 3000 50  0001 C CNN
 F 4 "160-1446-1-ND" H 0   0   50  0001 C CNN "Digi-Key PN"
