File: hdw/Logic_Board/LED_Display_Controller/Mechanical.sch (KiCad schematic (older format))
At the start: 36 parts

Commit message: Added some digikey partnumbers to components
Parts:
- MK3101, MK3102, MK3105, MK3106, MK3109, MK3110, MK3113, MK3114, MK3117, MK3118, MK3121, MK3122: Digi-Key PN (none) -> 36-8400-ND
- MK3103, MK3104, MK3107, MK3108, MK3111, MK3112, MK3115, MK3116, MK3119, MK3120, MK3123, MK3124: Digi-Key PN (none) -> 36-9900-ND
Changed lines of the file:
@@
 F 2 "" H 2520 2320 50  0001 C CNN
 F 3 "" H 2520 2320 50  0001 C CNN
+F 4 "36-8400-ND" H 0   0   50  0001 C CNN "Digi-Key PN"
 	1    2520 1970
 	1    0    0    -1
@@
 F 2 "" H 3520 2320 50  0001 C CNN
 F 3 "" H 3520 2320 50  0001 C CNN
+F 4 "36-8400-ND" H 0   0   50  0001 C CNN "Digi-Key PN"
 	1    3520 1970
 	1    0    0    -1
@@
 F 2 "" H 4520 2320 50  0001 C CNN
 F 3 "" H 4520 2320 50  0001 C CNN
+F 4 "36-8400-ND" H 0   0   50  0001 C CNN "Digi-Key PN"
 	1    4520 1970
 	1    0    0    -1
@@
 F 2 "" H 5520 2320 50  0001 C CNN
 F 3 "" H 5520 2320 50  0001 C CNN
+F 4 "36-8400-ND" H 0   0   50  0001 C CNN "Digi-Key PN"
 	1    5520 1970
 	1    0    0    -1
@@
 F 2 "" H 2520 3020 50  0001 C CNN
 F 3 "" H 2520 3020 50  0001 C CNN
+F 4 "36-8400-ND" H 0   0   50  0001 C CNN "Digi-Key PN"
 	1    2520 2670
 	1    0    0    -1
@@
 F 2 "" H 3520 3020 50  0001 C CNN
 F 3 "" H 3520 3020 50  0001 C CNN
+F 4 "36-8400-ND" H 0   0   50  0001 C CNN "Digi-Key PN"
 	1    3520 2670
 	1    0    0    -1
@@
 F 2 "" H 4520 3020 50  0001 C CNN
 F 3 "" H 4520 3020 50  0001 C CNN
+F 4 "36-8400-ND" H 0   0   50  0001 C CNN "Digi-Key PN"
 	1    4520 2670
 	1    0    0    -1
@@
 F 2 "" H 5520 3020 50  0001 C CNN
 F 3 "" H 5520 3020 50  0001 C CNN
+F 4 "36-8400-ND" H 0   0   50  0001 C CNN "Digi-Key PN"
 	1    5520 2670
 	1    0    0    -1
@@
 F 2 "" H 2520 3690 50  0001 C CNN
 F 3 "" H 2520 3690 50  0001 C CNN
+F 4 "36-9900-ND" H 0   0   50  0001 C CNN "Digi-Key PN"
 	1    2520 3440
 	1    0    0    -1
@@
 F 2 "" H 3520 3690 50  0001 C CNN
 F 3 "" H 3520 3690 50  0001 C CNN
+F 4 "36-9900-ND" H 0   0   50  0001 C CNN "Digi-Key PN"
 	1    3520 3440
 	1    0    0    -1
@@
 F 2 "" H 4520 3690 50  0001 C CNN
 F 3 "" H 4520 3690 50  0001 C CNN
+F 4 "36-9900-ND" H 0   0   50  0001 C CNN "Digi-Key PN"
 	1    4520 3440
 	1    0    0    -1
@@
 F 2 "" H 5520 3690 50  0001 C CNN
 F 3 "" H 5520 3690 50  0001 C CNN
+F 4 "36-9900-ND" H 0   0   50  0001 C CNN "Digi-Key PN"
 	1    5520 3440
 	1    0    0    -1
@@
 F 2 "" H 2520 4390 50  0001 C CNN
 F 3 "" H 2520 4390 50  0001 C CNN
+F 4 "36-9900-ND" H 0   0   50  0001 C CNN "Digi-Key PN"
 	1    2520 4140
 	1    0    0    -1
@@
 F 2 "" H 3520 4390 50  0001 C CNN
 F 3 "" H 3520 4390 50  0001 C CNN
+F 4 "36-9900-ND" H 0   0   50  0001 C CNN "Digi-Key PN"
 	1    3520 4140
 	1    0    0    -1
@@
 F 2 "" H 4520 4390 50  0001 C CNN
 F 3 "" H 4520 4390 50  0001 C CNN
+F 4 "36-9900-ND" H 0   0   50  0001 C CNN "Digi-Key PN"
 	1    4520 4140
 	1    0    0    -1
@@
 F 2 "" H 5520 4390 50  0001 C CNN
 F 3 "" H 5520 4390 50  0001 C CNN
+F 4 "36-9900-ND" H 0   0   50  0001 C CNN "Digi-Key PN"
 	1    5520 4140
 	1    0    0    -1
@@
 F 2 "" H 6520 2320 50  0001 C CNN
 F 3 "" H 6520 2320 50  0001 C CNN
+F 4 "36-8400-ND" H 0   0   50  0001 C CNN "Digi-Key PN"
 	1    6520 1970
 	1    0    0    -1
@@
 F 2 "" H 7520 2320 50  0001 C CNN
 F 3 "" H 7520 2320 50  0001 C CNN
+F 4 "36-8400-ND" H 0   0   50  0001 C CNN "Digi-Key PN"
 	1    7520 1970
 	1    0    0    -1
@@
 F 2 "" H 6520 3020 50  0001 C CNN
 F 3 "" H 6520 3020 50  0001 C CNN
+F 4 "36-8400-ND" H 0   0   50  0001 C CNN "Digi-Key PN"
 	1    6520 2670
 	1    0    0    -1
@@
 F 2 "" H 7520 3020 50  0001 C CNN
 F 3 "" H 7520 3020 50  0001 C CNN
+F 4 "36-8400-ND" H 0   0   50  0001 C CNN "Digi-Key PN"
 	1    7520 2670
 	1    0    0    -1
@@
 F 2 "" H 6520 3690 50  0001 C CNN
 F 3 "" H 6520 3690 50  0001 C CNN
+F 4 "36-9900-ND" H 0   0   50  0001 C CNN "Digi-Key PN"
 	1    6520 3440
 	1    0    0    -1
@@
 F 2 "" H 7520 3690 50  0001 C CNN
 F 3 "" H 7520 3690 50  0001 C CNN
+F 4 "36-9900-ND" H 0   0   50  0001 C CNN "Digi-Key PN"
 	1    7520 3440
 	1    0    0    -1
@@
 F 2 "" H 6520 4390 50  0001 C CNN
 F 3 "" H 6520 4390 50  0001 C CNN
+F 4 "36-9900-ND" H 0   0   50  0001 C CNN "Digi-Key PN"
 	1    6520 4140
 	1    0    0    -1
@@
 F 2 "" H 7520 4390 50  0001 C CNN
 F 3 "" H 7520 4390 50  0001 C CNN
+F 4 "36-9900-ND" H 0   0   50  0001 C CNN "Digi-Key PN"
 	1    7520 4140
 	1    0    0    -1

Commit message: First pass assignment of footprints to all components
Parts:
- H3101, H3102, H3103, H3104, H3105, H3106, H3107, H3108, H3109, H3110, H3111, H3112: footprint (none) -> Mounting_Holes:MountingHole_3mm_Pad_Via
Changed lines of the file:
@@
 F 0 "H3101" H 2520 4990 50  0000 C CNN
 F 1 "3mm Mounting Hole" H 2520 4915 50  0000 C CNN
-F 2 "" H 2520 4790 50  0001 C CNN
+F 2 "Mounting_Holes:MountingHole_3mm_Pad_Via" H 2520 4790 50  0001 C CNN
 F 3 "~" H 2520 4790 50  0001 C CNN
 	1    2520 4790
@@
 F 0 "H3103" H 3520 4990 50  0000 C CNN
 F 1 "3mm Mounting Hole" H 3520 4915 50  0000 C CNN
-F 2 "" H 3520 4790 50  0001 C CNN
+F 2 "Mounting_Holes:MountingHole_3mm_Pad_Via" H 3520 4790 50  0001 C CNN
 F 3 "~" H 3520 4790 50  0001 C CNN
 	1    3520 4790
@@
 F 0 "H3105" H 4520 4990 50  0000 C CNN
 F 1 "3mm Mounting Hole" H 4520 4915 50  0000 C CNN
-F 2 "" H 4520 4790 50  0001 C CNN
+F 2 "Mounting_Holes:MountingHole_3mm_Pad_Via" H 4520 4790 50  0001 C CNN
 F 3 "~" H 4520 4790 50  0001 C CNN
 	1    4520 4790
@@
 F 0 "H3107" H 5520 4990 50  0000 C CNN
 F 1 "3mm Mounting Hole" H 5520 4915 50  0000 C CNN
-F 2 "" H 5520 4790 50  0001 C CNN
+F 2 "Mounting_Holes:MountingHole_3mm_Pad_Via" H 5520 4790 50  0001 C CNN
 F 3 "~" H 5520 4790 50  0001 C CNN
 	1    5520 4790
@@
 F 0 "H3109" H 6520 4990 50  0000 C CNN
 F 1 "3mm Mounting Hole" H 6520 4915 50  0000 C CNN
-F 2 "" H 6520 4790 50  0001 C CNN
+F 2 "Mounting_Holes:MountingHole_3mm_Pad_Via" H 6520 4790 50  0001 C CNN
 F 3 "~" H 6520 4790 50  0001 C CNN
 	1    6520 4790
@@
 F 0 "H3111" H 7520 4990 50  0000 C CNN
 F 1 "3mm Mounting Hole" H 7520 4915 50  0000 C CNN
-F 2 "" H 7520 4790 50  0001 C CNN
+F 2 "Mounting_Holes:MountingHole_3mm_Pad_Via" H 7520 4790 50  0001 C CNN
 F 3 "~" H 7520 4790 50  0001 C CNN
 	1    7520 4790
@@
 F 0 "H3102" H 2520 5690 50  0000 C CNN
 F 1 "3mm Mounting Hole" H 2520 5615 50  0000 C CNN
-F 2 "" H 2520 5490 50  0001 C CNN
+F 2 "Mounting_Holes:MountingHole_3mm_Pad_Via" H 2520 5490 50  0001 C CNN
 F 3 "~" H 2520 5490 50  0001 C CNN
 	1    2520 5490
@@
 F 0 "H3104" H 3520 5690 50  0000 C CNN
 F 1 "3mm Mounting Hole" H 3520 5615 50  0000 C CNN
-F 2 "" H 3520 5490 50  0001 C CNN
+F 2 "Mounting_Holes:MountingHole_3mm_Pad_Via" H 3520 5490 50  0001 C CNN
 F 3 "~" H 3520 5490 50  0001 C CNN
 	1    3520 5490
@@
 F 0 "H3106" H 4520 5690 50  0000 C CNN
 F 1 "3mm Mounting Hole" H 4520 5615 50  0000 C CNN
-F 2 "" H 4520 5490 50  0001 C CNN
+F 2 "Mounting_Holes:MountingHole_3mm_Pad_Via" H 4520 5490 50  0001 C CNN
 F 3 "~" H 4520 5490 50  0001 C CNN
 	1    4520 5490
@@
 F 0 "H3108" H 5520 5690 50  0000 C CNN
 F 1 "3mm Mounting Hole" H 5520 5615 50  0000 C CNN
-F 2 "" H 5520 5490 50  0001 C CNN
+F 2 "Mounting_Holes:MountingHole_3mm_Pad_Via" H 5520 5490 50  0001 C CNN
 F 3 "~" H 5520 5490 50  0001 C CNN
 	1    5520 5490
@@
 F 0 "H3110" H 6520 5690 50  0000 C CNN
 F 1 "3mm Mounting Hole" H 6520 5615 50  0000 C CNN
-F 2 "" H 6520 5490 50  0001 C CNN
+F 2 "Mounting_Holes:MountingHole_3mm_Pad_Via" H 6520 5490 50  0001 C CNN
 F 3 "~" H 6520 5490 50  0001 C CNN
 	1    6520 5490
@@
 F 0 "H3112" H 7520 5690 50  0000 C CNN
 F 1 "3mm Mounting Hole" H 7520 5615 50  0000 C CNN
-F 2 "" H 7520 5490 50  0001 C CNN
+F 2 "Mounting_Holes:MountingHole_3mm_Pad_Via" H 7520 5490 50  0001 C CNN
 F 3 "~" H 7520 5490 50  0001 C CNN
 	1    7520 5490

Commit message: More routing
Parts:
- MK3101, MK3102, MK3105, MK3106, MK3109, MK3110, MK3113, MK3114, MK3117, MK3118, MK3121, MK3122: Digi-Key PN 36-8400-ND -> 36-2204-ND
Changed lines of the file:
@@
 F 2 "" H 2520 2320 50  0001 C CNN
 F 3 "" H 2520 2320 50  0001 C CNN
-F 4 "36-8400-ND" H 0   0   50  0001 C CNN "Digi-Key PN"
+F 4 "36-2204-ND" H 0   0   50  0001 C CNN "Digi-Key PN"
 	1    2520 1970
 	1    0    0    -1
@@
 F 2 "" H 3520 2320 50  0001 C CNN
 F 3 "" H 3520 2320 50  0001 C CNN
-F 4 "36-8400-ND" H 0   0   50  0001 C CNN "Digi-Key PN"
+F 4 "36-2204-ND" H 0   0   50  0001 C CNN "Digi-Key PN"
 	1    3520 1970
 	1    0    0    -1
@@
 F 2 "" H 4520 2320 50  0001 C CNN
 F 3 "" H 4520 2320 50  0001 C CNN
-F 4 "36-8400-ND" H 0   0   50  0001 C CNN "Digi-Key PN"
+F 4 "36-2204-ND" H 0   0   50  0001 C CNN "Digi-Key PN"
 	1    4520 1970
 	1    0    0    -1
@@
 F 2 "" H 5520 2320 50  0001 C CNN
 F 3 "" H 5520 2320 50  0001 C CNN
-F 4 "36-8400-ND" H 0   0   50  0001 C CNN "Digi-Key PN"
+F 4 "36-2204-ND" H 0   0   50  0001 C CNN "Digi-Key PN"
 	1    5520 1970
 	1    0    0    -1
@@
 F 2 "" H 2520 3020 50  0001 C CNN
 F 3 "" H 2520 3020 50  0001 C CNN
-F 4 "36-8400-ND" H 0   0   50  0001 C CNN "Digi-Key PN"
+F 4 "36-2204-ND" H 0   0   50  0001 C CNN "Digi-Key PN"
 	1    2520 2670
 	1    0    0    -1
@@
 F 2 "" H 3520 3020 50  0001 C CNN
 F 3 "" H 3520 3020 50  0001 C CNN
-F 4 "36-8400-ND" H 0   0   50  0001 C CNN "Digi-Key PN"
+F 4 "36-2204-ND" H 0   0   50  0001 C CNN "Digi-Key PN"
 	1    3520 2670
 	1    0    0    -1
@@
 F 2 "" H 4520 3020 50  0001 C CNN
 F 3 "" H 4520 3020 50  0001 C CNN
-F 4 "36-8400-ND" H 0   0   50  0001 C CNN "Digi-Key PN"
+F 4 "36-2204-ND" H 0   0   50  0001 C CNN "Digi-Key PN"
 	1    4520 2670
 	1    0    0    -1
@@
 F 2 "" H 5520 3020 50  0001 C CNN
 F 3 "" H 5520 3020 50  0001 C CNN
-F 4 "36-8400-ND" H 0   0   50  0001 C CNN "Digi-Key PN"
+F 4 "36-2204-ND" H 0   0   50  0001 C CNN "Digi-Key PN"
 	1    5520 2670
 	1    0    0    -1
@@
 F 2 "" H 6520 2320 50  0001 C CNN
 F 3 "" H 6520 2320 50  0001 C CNN
-F 4 "36-8400-ND" H 0   0   50  0001 C CNN "Digi-Key PN"
+F 4 "36-2204-ND" H 0   0   50  0001 C CNN "Digi-Key PN"
 	1    6520 1970
 	1    0    0    -1
@@
 F 2 "" H 6520 3020 50  0001 C CNN
 F 3 "" H 6520 3020 50  0001 C CNN
-F 4 "36-8400-ND" H 0   0   50  0001 C CNN "Digi-Key PN"
+F 4 "36-2204-ND" H 0   0   50  0001 C CNN "Digi-Key PN"
 	1    6520 2670
 	1    0    0    -1
@@
 F 2 "" H 7520 3020 50  0001 C CNN
 F 3 "" H 7520 3020 50  0001 C CNN
-F 4 "36-8400-ND" H 0   0   50  0001 C CNN "Digi-Key PN"
+F 4 "36-2204-ND" H 0   0   50  0001 C CNN "Digi-Key PN"
 	1    7520 2670
 	1    0    0    -1
@@
 F 2 "" H 7520 2320 50  0001 C CNN
 F 3 "" H 7520 2320 50  0001 C CNN
-F 4 "36-8400-ND" H 0   0   50  0001 C CNN "Digi-Key PN"
+F 4 "36-2204-ND" H 0   0   50  0001 C CNN "Digi-Key PN"
 	1    7520 1970
 	1    0    0    -1
